File: V3/kicad/4100_AddressBuffers.sch (KiCad schematic (older format))
At the start: 5 parts, among them U100 74LS541, U101 74LS541

Commit message: probably going to split into two boards
Parts:
- C100, C101: footprint (none) -> Capacitor_THT:C_Rect_L4.0mm_W2.5mm_P2.50mm
- U100, U101: footprint (none) -> Package_DIP:DIP-20_W7.62mm_LongPads
Changed lines of the file:
@@
 $Descr A4 11693 8268
 encoding utf-8
-Sheet 14 16
+Sheet 8 10
 Title ""
 Date ""
@@
 F 0 "U4100" H 5400 3281 50  0000 R CNN
 F 1 "74LS541" H 5400 3190 50  0000 R CNN
-F 2 "" H 5400 2300 50  0001 C CNN
+F 2 "Package_DIP:DIP-20_W7.62mm_LongPads" H 5400 2300 50  0001 C CNN
 F 3 "http://www.ti.com/lit/gpn/sn74LS541" H 5400 2300 50  0001 C CNN
 	1    5400 2300
@@
 F 0 "U4101" H 2900 3281 50  0000 R CNN
 F 1 "74LS541" H 2900 3190 50  0000 R CNN
-F 2 "" H 2900 2300 50  0001 C CNN
+F 2 "Package_DIP:DIP-20_W7.62mm_LongPads" H 2900 2300 50  0001 C CNN
 F 3 "http://www.ti.com/lit/gpn/sn74LS541" H 2900 2300 50  0001 C CNN
 	1    2900 2300
@@
 F 0 "C4100" H 8615 2246 50  0000 L CNN
 F 1 "C" H 8615 2155 50  0000 L CNN
-F 2 "" H 8538 2050 50  0001 C CNN
+F 2 "Capacitor_THT:C_Rect_L4.0mm_W2.5mm_P2.50mm" H 8538 2050 50  0001 C CNN
 F 3 "~" H 8500 2200 50  0001 C CNN
 	1    8500 2200
@@
 F 0 "C4101" H 9115 2246 50  0000 L CNN
 F 1 "C" H 9115 2155 50  0000 L CNN
-F 2 "" H 9038 2050 50  0001 C CNN
+F 2 "Capacitor_THT:C_Rect_L4.0mm_W2.5mm_P2.50mm" H 9038 2050 50  0001 C CNN
 F 3 "~" H 9000 2200 50  0001 C CNN
 	1    9000 2200
