File: V3/kicad/4200_CounterLogic.sch (KiCad schematic (older format))
At the start: 10 parts, among them U600 4040, U601 GAL16V8, U602 4040, U603 GAL16V8, X600 ACO-20.000MHz

Commit message: probably going to split into two boards
Parts:
- C600, C601, C602, C603, C604: footprint (none) -> Capacitor_THT:C_Rect_L4.0mm_W2.5mm_P2.50mm
- U600, U602: footprint (none) -> Package_DIP:DIP-16_W7.62mm_LongPads
- U601, U603: footprint (none) -> Package_DIP:DIP-20_W7.62mm_Socket_LongPads
Connections:
- net +5V: now also U600.16 (VDD), U601.20 (VCC), U602.16 (VDD), U603.20 (VCC)
- net H_CNT_RST renamed H_RST
- net H_CPU_EN renamed H_VIS
- net V_CNT_RST renamed V_RST
Other:
- note added: "0 - 399 Visible Area (Video Enable)\n400 - 419 Front Porch\n420 - 483 Pulse = (PC7 & C8 & (C6 | C5))\n484 - 527 Back Porch\n\n(Clock is 40MHz/2 so all values are 1/2\nAll values are divisible by 4 so that makes it even easier\n\nReset still needs all lines for most accurate signal\n\nH_VIS signals that the visible area has passed\nH_RST resets the 4040 count"
- note added: "0 - 599 Visible Area\n600 Front Porch\n601 - 604 Pulse\n605 - 627 Back Porch\n\nH_VIS + lines past the visible area = CPU_EN"
- note removed: "0 - 399 Visible Area (Video Enable)\n400 - 419 Front Porch\n420 - 483 Pulse = (PC7 & C8 & (C6 | C5))\n484 - 527 Back Porch\n\n(Clock is 40MHz/2 so all values are 1/2\nAll values are divisible by 4 so that makes it even easier\n\nReset still needs all lines for most accurate signal\n\nH_CPU_EN signals that the visible area has passed\nH_CNT_RST resets the 4040"
- note removed: "0 - 599 Visible Area\n600 Front Porch\n601 - 604 Pulse\n605 - 627 Back Porch\n\nH_CLU_EN + lines past the visible area = CPU_EN"
- moved on the sheet: X4200
