File: V3/kicad/4300_VideoOut.sch (KiCad schematic (older format))
At the start: 11 parts, among them J4300 DB15_Female_HighDensity_Mount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, SW4300 SW_DIP_x06, U4300 74LS151

Commit message: probably going to split into two boards
Parts:
- C4300: footprint (none) -> Capacitor_THT:C_Rect_L4.0mm_W2.5mm_P2.50mm
- JP4300: footprint (none) -> Connector_PinHeader_2.54mm:PinHeader_1x03_P2.54mm_Vertical
- U4300: footprint (none) -> Package_DIP:DIP-16_W7.62mm_LongPads
Changed lines of the file:
@@
 $Descr A4 11693 8268
 encoding utf-8
-Sheet 13 16
+Sheet 7 10
 Title ""
 Date ""
@@
 F 0 "U4300" H 3900 5181 50  0000 R CNN
 F 1 "74LS151" H 3900 5090 50  0000 R CNN
-F 2 "" H 3900 4100 50  0001 C CNN
+F 2 "Package_DIP:DIP-16_W7.62mm_LongPads" H 3900 4100 50  0001 C CNN
 F 3 "http://www.ti.com/lit/gpn/sn74LS151" H 3900 4100 50  0001 C CNN
 	1    3900 4100
@@
 F 0 "JP4300" H 6050 3789 50  0000 C CNN
 F 1 "Jumper_NC_Dual" H 6050 3698 50  0000 C CNN
-F 2 "" H 6050 3550 50  0001 C CNN
+F 2 "Connector_PinHeader_2.54mm:PinHeader_1x03_P2.54mm_Vertical" H 6050 3550 50  0001 C CNN
 F 3 "~" H 6050 3550 50  0001 C CNN
 	1    6050 3550
@@
 F 0 "C4300" H 5265 5196 50  0000 L CNN
 F 1 "C" H 5265 5105 50  0000 L CNN
-F 2 "" H 5188 5000 50  0001 C CNN
+F 2 "Capacitor_THT:C_Rect_L4.0mm_W2.5mm_P2.50mm" H 5188 5000 50  0001 C CNN
 F 3 "~" H 5150 5150 50  0001 C CNN
 	1    5150 5150
