File: V3/kicad/2300_Reset.sch (KiCad schematic (older format))
At the start: 7 parts, among them SW1000 SW_Push, U1000 LM555xM

Commit message: Updated PCB files
Changed lines of the file:
@@
 $Descr A4 11693 8268
 encoding utf-8
-Sheet 2 6
+Sheet 6 6
 Title ""
 Date ""
@@
 AR Path="/62497D60/624C743E" Ref="U?"  Part="1"
 AR Path="/61D852D7/624C743E" Ref="U1000"  Part="1"
-F 0 "U1000" H 5800 4631 50  0000 L TNN
+AR Path="/6191B6A2/624CF3AF/624C743E" Ref="U?"  Part="1"
+F 0 "U?" H 5800 4631 50  0000 L TNN
 F 1 "LM555xM" H 5800 4540 50  0000 L TNN
 F 2 "Package_DIP:DIP-8_W7.62mm_LongPads" H 6650 3650 50  0001 C CNN
@@
 AR Path="/62497D60/624C7444" Ref="#PWR?"  Part="1"
 AR Path="/61D852D7/624C7444" Ref="#PWR0101"  Part="1"
-F 0 "#PWR0101" H 5800 4450 50  0001 C CNN
+AR Path="/6191B6A2/624CF3AF/624C7444" Ref="#PWR?"  Part="1"
+F 0 "#PWR?" H 5800 4450 50  0001 C CNN
 F 1 "GND" H 5805 4527 50  0000 C CNN
 F 2 "" H 5800 4700 50  0001 C CNN
@@
 AR Path="/62497D60/624C744A" Ref="SW?"  Part="1"
 AR Path="/61D852D7/624C744A" Ref="SW1000"  Part="1"
-F 0 "SW1000" H 4350 4135 50  0000 C CNN
+AR Path="/6191B6A2/624CF3AF/624C744A" Ref="SW?"  Part="1"
+F 0 "SW?" H 4350 4135 50  0000 C CNN
 F 1 "SW_Push" H 4350 4044 50  0000 C CNN
 F 2 "Button_Switch_THT:SW_PUSH_6mm" H 4350 4050 50  0001 C CNN
@@
 AR Path="/62497D60/624C7456" Ref="C?"  Part="1"
 AR Path="/61D852D7/624C7456" Ref="C1001"  Part="1"
-F 0 "C1001" H 5115 4596 50  0000 L CNN
+AR Path="/6191B6A2/624CF3AF/624C7456" Ref="C?"  Part="1"
+F 0 "C?" H 5115 4596 50  0000 L CNN
 F 1 "C" H 5115 4505 50  0000 L CNN
 F 2 "Capacitor_THT:C_Rect_L4.0mm_W2.5mm_P2.50mm" H 5038 4400 50  0001 C CNN
@@
 AR Path="/62497D60/624C7467" Ref="C?"  Part="1"
 AR Path="/61D852D7/624C7467" Ref="C1002"  Part="1"
-F 0 "C1002" H 6815 4596 50  0000 L CNN
+AR Path="/6191B6A2/624CF3AF/624C7467" Ref="C?"  Part="1"
+F 0 "C?" H 6815 4596 50  0000 L CNN
 F 1 "C" H 6815 4505 50  0000 L CNN
 F 2 "Capacitor_THT:C_Rect_L4.0mm_W2.5mm_P2.50mm" H 6738 4400 50  0001 C CNN
@@
 U 1 1 625B99BC
 P 7900 3900
-F 0 "C1000" H 8015 3946 50  0000 L CNN
+AR Path="/61D852D7/625B99BC" Ref="C1000"  Part="1"
+AR Path="/6191B6A2/624CF3AF/625B99BC" Ref="C?"  Part="1"
+F 0 "C?" H 8015 3946 50  0000 L CNN
 F 1 "C" H 8015 3855 50  0000 L CNN
 F 2 "Capacitor_THT:C_Rect_L4.0mm_W2.5mm_P2.50mm" H 7938 3750 50  0001 C CNN
@@
 AR Path="/62497D60/625BC077" Ref="#PWR?"  Part="1"
 AR Path="/61D852D7/625BC077" Ref="#PWR0102"  Part="1"
-F 0 "#PWR0102" H 7900 3800 50  0001 C CNN
+AR Path="/6191B6A2/624CF3AF/625BC077" Ref="#PWR?"  Part="1"
+F 0 "#PWR?" H 7900 3800 50  0001 C CNN
 F 1 "GND" H 7905 3877 50  0000 C CNN
 F 2 "" H 7900 4050 50  0001 C CNN
@@
 AR Path="/62497D60/62633FFA" Ref="C?"  Part="1"
 AR Path="/61D852D7/62633FFA" Ref="C1003"  Part="1"
-F 0 "C1003" H 4665 4596 50  0000 L CNN
+AR Path="/6191B6A2/624CF3AF/62633FFA" Ref="C?"  Part="1"
+F 0 "C?" H 4665 4596 50  0000 L CNN
 F 1 "C" H 4665 4505 50  0000 L CNN
 F 2 "Capacitor_THT:C_Rect_L4.0mm_W2.5mm_P2.50mm" H 4588 4400 50  0001 C CNN
@@
 U 1 1 61A98508
 P 5900 2300
-F 0 "RN1000" H 6088 2346 50  0000 L CNN
+AR Path="/61D852D7/61A98508" Ref="RN1000"  Part="1"
+AR Path="/6191B6A2/624CF3AF/61A98508" Ref="RN?"  Part="1"
+F 0 "RN?" H 6088 2346 50  0000 L CNN
 F 1 "R_Network04" H 6088 2255 50  0000 L CNN
 F 2 "Resistor_THT:R_Array_SIP5" V 6175 2300 50  0001 C CNN
@@
 U 1 1 61E872A1
 P 5700 2100
-F 0 "#PWR0103" H 5700 1950 50  0001 C CNN
+AR Path="/61D852D7/61E872A1" Ref="#PWR0103"  Part="1"
+AR Path="/6191B6A2/624CF3AF/61E872A1" Ref="#PWR?"  Part="1"
+F 0 "#PWR?" H 5700 1950 50  0001 C CNN
 F 1 "+5V" V 5715 2228 50  0000 L CNN
 F 2 "" H 5700 2100 50  0001 C CNN
@@
 U 1 1 61E87BC4
 P 5800 3350
-F 0 "#PWR0104" H 5800 3200 50  0001 C CNN
+AR Path="/61D852D7/61E87BC4" Ref="#PWR0104"  Part="1"
+AR Path="/6191B6A2/624CF3AF/61E87BC4" Ref="#PWR?"  Part="1"
+F 0 "#PWR?" H 5800 3200 50  0001 C CNN
 F 1 "+5V" V 5815 3478 50  0000 L CNN
 F 2 "" H 5800 3350 50  0001 C CNN
@@
 U 1 1 61E8CD41
 P 7900 3750
-F 0 "#PWR0105" H 7900 3600 50  0001 C CNN
+AR Path="/61D852D7/61E8CD41" Ref="#PWR0105"  Part="1"
+AR Path="/6191B6A2/624CF3AF/61E8CD41" Ref="#PWR?"  Part="1"
+F 0 "#PWR?" H 7900 3600 50  0001 C CNN
 F 1 "+5V" V 7915 3878 50  0000 L CNN
 F 2 "" H 7900 3750 50  0001 C CNN
@@
 U 1 1 620357A9
 P 5300 4250
-F 0 "#PWR0106" H 5300 4100 50  0001 C CNN
+AR Path="/61D852D7/620357A9" Ref="#PWR0106"  Part="1"
+AR Path="/6191B6A2/624CF3AF/620357A9" Ref="#PWR?"  Part="1"
+F 0 "#PWR?" H 5300 4100 50  0001 C CNN
 F 1 "+5V" V 5315 4378 50  0000 L CNN
 F 2 "" H 5300 4250 50  0001 C CNN
