File: V3/kicad/_autosave-2100_ALTCPU.sch (KiCad schematic (older format))
At the start: 7 parts, among them J2100 Conn_02x20_Counter_Clockwise, U2100 Z8-L180-S180-180-PQFP-80, U2101 GAL16V8, X2100 14.7456 MHz

Commit message: fixing up CPU page and routing
Other:
- note added: "RTS0 defaults to 1 and can be controlled via internal registers\nSetting it low disables part of the ROM window"
- note removed: "RTS0 defaults to 1 and can be controlled via internal registers\nSetting it low disables the ROM window"
Changed lines of the file:
@@
 	2000 6350 1750 6350
 Text Notes 1450 7600 0    50   ~ 0
-RTS0 defaults to 1 and can be controlled via internal registers\nSetting it low disables the ROM window
+RTS0 defaults to 1 and can be controlled via internal registers\nSetting it low disables part of the ROM window
 Wire Wire Line
 	3600 6650 3000 6650
@@
 DREQ0
 $Comp
-L power:GND #PWR?
+L power:GND #PWR0140
 U 1 1 6275CB20
 P 2100 3750
-F 0 "#PWR?" H 2100 3500 50  0001 C CNN
+F 0 "#PWR0140" H 2100 3500 50  0001 C CNN
 F 1 "GND" H 2105 3577 50  0000 C CNN
 F 2 "" H 2100 3750 50  0001 C CNN
@@
 $EndComp
 $Comp
-L power:+5V #PWR?
+L power:+5V #PWR0142
 U 1 1 6275CB26
 P 2100 1850
-F 0 "#PWR?" H 2100 1700 50  0001 C CNN
+F 0 "#PWR0142" H 2100 1700 50  0001 C CNN
 F 1 "+5V" V 2115 1978 50  0000 L CNN
 F 2 "" H 2100 1850 50  0001 C CNN
@@
 $EndComp
 $Comp
-L power:+5V #PWR?
+L power:+5V #PWR0144
 U 1 1 627A29E2
 P 2100 1950
-F 0 "#PWR?" H 2100 1800 50  0001 C CNN
+F 0 "#PWR0144" H 2100 1800 50  0001 C CNN
 F 1 "+5V" V 2115 2078 50  0000 L CNN
 F 2 "" H 2100 1950 50  0001 C CNN
