File: V3/kicad/2210_SD_Card.sch (KiCad schematic (older format))
At the start: 7 parts, among them J2210 Micro_SD_Card_Det, U2210 74LS07, U2213 TL760M33

Commit message: last touches on peripherals and memory
Parts:
- added unit 6 of U2210
Connections:
- net +3V3: no longer U2210.11
- net +5V: now also U2210.11, U2210.13
- no-connect marks 2 -> 4
Other:
- note removed: "probably HC or HCT, not LS for 3.3"
- moved on the sheet: RN2210, U2210C
Changed lines of the file:
@@
 	1    0    0    -1
 $EndComp
-Text Notes 6600 3850 0    50   ~ 0
-probably HC or HCT, not LS for 3.3
 NoConn ~ 6150 2650
 NoConn ~ 6150 3350
@@
 $EndComp
 Wire Wire Line
-	5800 3250 6150 3250
+	5000 3750 4650 3750
 $Comp
 L power:+3.3V #PWR?
@@
 	0    -1   -1   0
 $EndComp
+Text Label 8100 4700 0    50   ~ 0
+SD_SCK
+Text Label 8100 4800 0    50   ~ 0
+SD_MOSI
+Wire Wire Line
+	8100 4700 8450 4700
+Wire Wire Line
+	8100 4800 8450 4800
+Wire Wire Line
+	8450 4500 8100 4500
 Text Label 8100 4500 0    50   ~ 0
-SD_SCK
+SD_CS
 Text Label 8100 4600 0    50   ~ 0
-SD_MOSI
-Wire Wire Line
-	8100 4500 8450 4500
+SD_MISO
 Wire Wire Line
 	8100 4600 8450 4600
-Wire Wire Line
-	8450 4300 8100 4300
-Text Label 8100 4300 0    50   ~ 0
-SD_CS
-Text Label 8100 4400 0    50   ~ 0
-SD_MISO
-Wire Wire Line
-	8100 4400 8450 4400
 $Comp
 L power:+3.3V #PWR?
 U 1 1 6259F3FB
-P 8850 4300
+P 8850 4500
 AR Path="/6191B6A2/61F28B7D/6259F3FB" Ref="#PWR?"  Part="1"
 AR Path="/6191B6A2/61F28B7D/62590ED9/6259F3FB" Ref="#PWR0117"  Part="1"
-F 0 "#PWR0117" H 8850 4150 50  0001 C CNN
-F 1 "+3.3V" V 8865 4428 50  0000 L CNN
-F 2 "" H 8850 4300 50  0001 C CNN
-F 3 "" H 8850 4300 50  0001 C CNN
-	1    8850 4300
+F 0 "#PWR0117" H 8850 4350 50  0001 C CNN
+F 1 "+3.3V" V 8865 4628 50  0000 L CNN
+F 2 "" H 8850 4500 50  0001 C CNN
+F 3 "" H 8850 4500 50  0001 C CNN
+	1    8850 4500
 	0    1    1    0
 $EndComp
@@
 AR Path="/6191B6A2/61F28B7D/625A5E8B" Ref="U?"  Part="1"
 AR Path="/6191B6A2/61F28B7D/62590ED9/625A5E8B" Ref="U2210"  Part="1"
-F 0 "U2210" H 4350 3117 50  0000 C CNN
-F 1 "74LS07" H 4350 3026 50  0000 C CNN
+F 0 "U2210" H 3500 2900 50  0000 C CNN
+F 1 "74LS07" H 3500 2800 50  0000 C CNN
 F 2 "Package_SO:SOIC-14_3.9x8.7mm_P1.27mm" H 4350 2800 50  0001 C CNN
 F 3 "www.ti.com/lit/ds/symlink/sn74ls07.pdf" H 4350 2800 50  0001 C CNN
@@
 AR Path="/6191B6A2/61F28B7D/625A5E91" Ref="U?"  Part="2"
 AR Path="/6191B6A2/61F28B7D/62590ED9/625A5E91" Ref="U2210"  Part="2"
-F 0 "U2210" H 4350 3617 50  0000 C CNN
-F 1 "74LS07" H 4350 3526 50  0000 C CNN
+F 0 "U2210" H 3500 3400 50  0000 C CNN
+F 1 "74LS07" H 3500 3300 50  0000 C CNN
 F 2 "Package_SO:SOIC-14_3.9x8.7mm_P1.27mm" H 4350 3300 50  0001 C CNN
 F 3 "www.ti.com/lit/ds/symlink/sn74ls07.pdf" H 4350 3300 50  0001 C CNN
@@
 L 74xx:74LS07 U?
 U 3 1 625A5E97
-P 4350 3600
+P 4350 3750
 AR Path="/6191B6A2/61F28B7D/625A5E97" Ref="U?"  Part="3"
 AR Path="/6191B6A2/61F28B7D/62590ED9/625A5E97" Ref="U2210"  Part="3"
-F 0 "U2210" H 4350 3917 50  0000 C CNN
-F 1 "74LS07" H 4350 3826 50  0000 C CNN
-F 2 "Package_SO:SOIC-14_3.9x8.7mm_P1.27mm" H 4350 3600 50  0001 C CNN
-F 3 "www.ti.com/lit/ds/symlink/sn74ls07.pdf" H 4350 3600 50  0001 C CNN
-	3    4350 3600
+F 0 "U2210" H 5200 3800 50  0000 C CNN
+F 1 "74LS07" H 5200 3700 50  0000 C CNN
+F 2 "Package_SO:SOIC-14_3.9x8.7mm_P1.27mm" H 4350 3750 50  0001 C CNN
+F 3 "www.ti.com/lit/ds/symlink/sn74ls07.pdf" H 4350 3750 50  0001 C CNN
+	3    4350 3750
 	-1   0    0    1
 $EndComp
@@
 AR Path="/6191B6A2/61F28B7D/625A5E9D" Ref="U?"  Part="4"
 AR Path="/6191B6A2/61F28B7D/62590ED9/625A5E9D" Ref="U2210"  Part="4"
-F 0 "U2210" H 4350 2617 50  0000 C CNN
-F 1 "74LS07" H 4350 2526 50  0000 C CNN
+F 0 "U2210" H 3500 2400 50  0000 C CNN
+F 1 "74LS07" H 3500 2300 50  0000 C CNN
 F 2 "Package_SO:SOIC-14_3.9x8.7mm_P1.27mm" H 4350 2300 50  0001 C CNN
 F 3 "www.ti.com/lit/ds/symlink/sn74ls07.pdf" H 4350 2300 50  0001 C CNN
@@
 AR Path="/6191B6A2/61F28B7D/625A5EA9" Ref="U?"  Part="7"
 AR Path="/6191B6A2/61F28B7D/62590ED9/625A5EA9" Ref="U2210"  Part="7"
-F 0 "U2210" H 4730 4696 50  0000 L CNN
-F 1 "74LS07" H 4730 4605 50  0000 L CNN
+F 0 "U2210" V 4900 4550 50  0000 L CNN
+F 1 "74LS07" V 4800 4550 50  0000 L CNN
 F 2 "Package_SO:SOIC-14_3.9x8.7mm_P1.27mm" H 4500 4650 50  0001 C CNN
 F 3 "www.ti.com/lit/ds/symlink/sn74ls07.pdf" H 4500 4650 50  0001 C CNN
@@
 $EndComp
 Wire Wire Line
-	5000 3300 4650 3300
-Wire Wire Line
-	5000 2800 4650 2800
-Wire Wire Line
-	5000 2850 5000 2800
-Wire Wire Line
-	5000 2850 6150 2850
-Wire Wire Line
-	5000 3300 5000 3050
-Wire Wire Line
-	5000 3050 6150 3050
-Wire Wire Line
-	5800 3600 5800 3250
-Wire Wire Line
-	4650 3600 5800 3600
+	4650 3300 5000 3300
+Wire Wire Line
+	4650 2800 5000 2800
 $Comp
 L power:+5V #PWR?
@@
 	0    -1   -1   0
 $EndComp
-Wire Wire Line
-	5400 2750 5400 2300
-Wire Wire Line
-	5400 2750 6150 2750
-Wire Wire Line
-	4650 2300 5400 2300
 Text HLabel 4050 2300 0    50   Input ~ 0
 CS
@@
 Text HLabel 4050 3300 0    50   Input ~ 0
 SCK
-Text HLabel 4050 3600 0    50   Output ~ 0
+Text HLabel 4050 3750 0    50   Output ~ 0
 MISO
-Text Label 5800 2750 0    50   ~ 0
+Text Label 5000 2300 2    50   ~ 0
 SD_CS
-Text Label 5800 2850 0    50   ~ 0
+Text Label 5000 2800 2    50   ~ 0
 SD_MOSI
-Text Label 5800 3050 0    50   ~ 0
+Text Label 5000 3300 2    50   ~ 0
 SD_SCK
-Text Label 5800 3250 0    50   ~ 0
+Text Label 5000 3750 2    50   ~ 0
 SD_MISO
 Text Notes 7800 6900 0    118  ~ 24
@@
 L Device:R_Network05 RN2210
 U 1 1 62618FEB
-P 8650 4500
-F 0 "RN2210" V 8233 4500 50  0000 C CNN
-F 1 "10k" V 8324 4500 50  0000 C CNN
-F 2 "Resistor_THT:R_Array_SIP6" V 9025 4500 50  0001 C CNN
-F 3 "http://www.vishay.com/docs/31509/csc.pdf" H 8650 4500 50  0001 C CNN
-	1    8650 4500
-	0    1    1    0
-$EndComp
-$Comp
-L power:+3.3V #PWR?
-U 1 1 626AA2AE
+P 8650 4700
+F 0 "RN2210" V 8233 4700 50  0000 C CNN
+F 1 "10k" V 8324 4700 50  0000 C CNN
+F 2 "Resistor_THT:R_Array_SIP6" V 9025 4700 50  0001 C CNN
+F 3 "http://www.vishay.com/docs/31509/csc.pdf" H 8650 4700 50  0001 C CNN
+	1    8650 4700
+	0    1    1    0
+$EndComp
+Wire Wire Line
+	5800 3250 6150 3250
+Text Label 5800 3250 0    50   ~ 0
+SD_MISO
+Wire Wire Line
+	6150 3050 5800 3050
+Text Label 5800 3050 0    50   ~ 0
+SD_SCK
+Wire Wire Line
+	6150 2850 5800 2850
+Text Label 5800 2850 0    50   ~ 0
+SD_MOSI
+Text Label 5800 2750 0    50   ~ 0
+SD_CS
+Wire Wire Line
+	5800 2750 6150 2750
+Wire Wire Line
+	4650 2300 5000 2300
+$Comp
+L 74xx:74LS07 U2210
+U 6 1 6293BD1C
+P 3450 5200
+F 0 "U2210" H 3450 5500 50  0000 C CNN
+F 1 "74LS07" H 3450 5400 50  0000 C CNN
+F 2 "Package_SO:SOIC-14_3.9x8.7mm_P1.27mm" H 3450 5200 50  0001 C CNN
+F 3 "www.ti.com/lit/ds/symlink/sn74ls07.pdf" H 3450 5200 50  0001 C CNN
+	6    3450 5200
+	-1   0    0    1
+$EndComp
+$Comp
+L power:+5V #PWR?
+U 1 1 6293E9E7
+P 3750 5200
+AR Path="/6191B6A2/61F28B7D/6293E9E7" Ref="#PWR?"  Part="1"
+AR Path="/6191B6A2/61F28B7D/62590ED9/6293E9E7" Ref="#PWR?"  Part="1"
+F 0 "#PWR?" H 3750 5050 50  0001 C CNN
+F 1 "+5V" V 3765 5328 50  0000 L CNN
+F 2 "" H 3750 5200 50  0001 C CNN
+F 3 "" H 3750 5200 50  0001 C CNN
+	1    3750 5200
+	0    1    1    0
+$EndComp
+$Comp
+L power:+5V #PWR?
+U 1 1 6293F178
 P 4800 5200
-AR Path="/6191B6A2/61F28B7D/626AA2AE" Ref="#PWR?"  Part="1"
-AR Path="/6191B6A2/61F28B7D/62590ED9/626AA2AE" Ref="#PWR0123"  Part="1"
-F 0 "#PWR0123" H 4800 5050 50  0001 C CNN
-F 1 "+3.3V" V 4815 5328 50  0000 L CNN
+AR Path="/6191B6A2/61F28B7D/6293F178" Ref="#PWR?"  Part="1"
+AR Path="/6191B6A2/61F28B7D/62590ED9/6293F178" Ref="#PWR?"  Part="1"
+F 0 "#PWR?" H 4800 5050 50  0001 C CNN
+F 1 "+5V" V 4815 5328 50  0000 L CNN
 F 2 "" H 4800 5200 50  0001 C CNN
 F 3 "" H 4800 5200 50  0001 C CNN
@@
 	0    1    1    0
 $EndComp
+NoConn ~ 4200 5200
+NoConn ~ 3150 5200
 $EndSCHEMATC
