File: V3/kicad/2210_SD_Card.sch (KiCad schematic (older format))
At the start: 7 parts, among them J2210 Micro_SD_Card_Det, U2210 74LS07, U2213 TL760M33

Commit message: minor changes to make routing easier
Changed lines of the file:
@@
-	0    1    1    0
-$EndComp
-$Comp
-L power:+5V #PWR?
-U 1 1 6293F178
-P 4800 5200
-AR Path="/6191B6A2/61F28B7D/6293F178" Ref="#PWR?"  Part="1"
-AR Path="/6191B6A2/61F28B7D/62590ED9/6293F178" Ref="#PWR0166"  Part="1"
-F 0 "#PWR0166" H 4800 5050 50  0001 C CNN
-F 1 "+5V" V 4815 5328 50  0000 L CNN
-F 2 "" H 4800 5200 50  0001 C CNN
-F 3 "" H 4800 5200 50  0001 C CNN
-	1    4800 5200
 	0    1    1    0
 $EndComp
 NoConn ~ 4200 5200
 NoConn ~ 3150 5200
+$Comp
+L power:GND #PWR?
+U 1 1 6281E96A
+P 4800 5200
+AR Path="/6191B6A2/61F28B7D/6281E96A" Ref="#PWR?"  Part="1"
+AR Path="/6191B6A2/61F28B7D/62590ED9/6281E96A" Ref="#PWR?"  Part="1"
+F 0 "#PWR?" H 4800 4950 50  0001 C CNN
+F 1 "GND" H 4805 5027 50  0000 C CNN
+F 2 "" H 4800 5200 50  0001 C CNN
+F 3 "" H 4800 5200 50  0001 C CNN
+	1    4800 5200
+	0    -1   -1   0
+$EndComp
 $EndSCHEMATC

Commit message: Completely redesigned board layout
Parts:
- removed C2213A1: .1uF, Capacitor_THT:CP_Radial_D5.0mm_P2.00mm, symbol Device:CP1
- removed C22213B1: 22uF, Capacitor_THT:CP_Radial_D5.0mm_P2.00mm, symbol Device:CP1
- removed U2213: TL760M33, Package_TO_SOT_SMD:TO-252-3_TabPin2, symbol Regulator_Linear:LD39150DT33
Connections:
- net labels removed: VCC
- wire segments 20 -> 14
Changed lines of the file:
@@
 $EndComp
-$Comp
-L Regulator_Linear:LD39150DT33 U?
-U 1 1 6259F407
-P 6800 4550
-AR Path="/6191B6A2/61F28B7D/6259F407" Ref="U?"  Part="1"
-AR Path="/6191B6A2/61F28B7D/62590ED9/6259F407" Ref="U2213"  Part="1"
-F 0 "U2213" H 6800 4792 50  0000 C CNN
-F 1 "TL760M33" H 6800 4701 50  0000 C CNN
-F 2 "Package_TO_SOT_SMD:TO-252-3_TabPin2" H 6800 4750 50  0001 C CNN
-F 3 "https://www.st.com/resource/en/datasheet/ld39150.pdf" H 6900 4300 50  0001 C CNN
-	1    6800 4550
-	1    0    0    -1
-$EndComp
-$Comp
-L power:+3.3V #PWR?
-U 1 1 6259F413
-P 7200 4550
-AR Path="/6191B6A2/61F28B7D/6259F413" Ref="#PWR?"  Part="1"
-AR Path="/6191B6A2/61F28B7D/62590ED9/6259F413" Ref="#PWR0120"  Part="1"
-F 0 "#PWR0120" H 7200 4400 50  0001 C CNN
-F 1 "+3.3V" V 7215 4678 50  0000 L CNN
-F 2 "" H 7200 4550 50  0001 C CNN
-F 3 "" H 7200 4550 50  0001 C CNN
-	1    7200 4550
-	0    1    1    0
-$EndComp
-$Comp
-L power:GND #PWR?
-U 1 1 6259F419
-P 6800 4850
-AR Path="/6191B6A2/61F28B7D/6259F419" Ref="#PWR?"  Part="1"
-AR Path="/6191B6A2/61F28B7D/62590ED9/6259F419" Ref="#PWR0124"  Part="1"
-F 0 "#PWR0124" H 6800 4600 50  0001 C CNN
-F 1 "GND" H 6805 4677 50  0000 C CNN
-F 2 "" H 6800 4850 50  0001 C CNN
-F 3 "" H 6800 4850 50  0001 C CNN
-	1    6800 4850
-	1    0    0    -1
-$EndComp
-Wire Wire Line
-	6450 4850 6800 4850
-Wire Wire Line
-	6800 4850 7150 4850
-Connection ~ 6800 4850
 $Comp
 L 74xx:74LS07 U?
@@
 This page has been checked!
 $Comp
-L power:VCC #PWR0143
-U 1 1 62567B69
-P 6400 4550
-F 0 "#PWR0143" H 6400 4400 50  0001 C CNN
-F 1 "VCC" V 6415 4677 50  0000 L CNN
-F 2 "" H 6400 4550 50  0001 C CNN
-F 3 "" H 6400 4550 50  0001 C CNN
-	1    6400 4550
-	0    -1   -1   0
-$EndComp
-$Comp
 L Device:C C?
 U 1 1 62613B08
@@
 $EndComp
 $Comp
-L Device:CP1 C?
-U 1 1 6261578C
-P 7150 4700
-AR Path="/6261578C" Ref="C?"  Part="1"
-AR Path="/6191B6A2/61F28B7D/62590ED9/6261578C" Ref="C22213B1"  Part="1"
-F 0 "C22213B1" H 7265 4746 50  0000 L CNN
-F 1 "22uF" H 7265 4655 50  0000 L CNN
-F 2 "Capacitor_THT:CP_Radial_D5.0mm_P2.00mm" H 7150 4700 50  0001 C CNN
-F 3 "~" H 7150 4700 50  0001 C CNN
-	1    7150 4700
-	1    0    0    -1
-$EndComp
-Wire Wire Line
-	7100 4550 7150 4550
-Wire Wire Line
-	6400 4550 6450 4550
-$Comp
-L Device:CP1 C?
-U 1 1 626150D9
-P 6450 4700
-AR Path="/626150D9" Ref="C?"  Part="1"
-AR Path="/6191B6A2/61F28B7D/62590ED9/626150D9" Ref="C2213A1"  Part="1"
-F 0 "C2213A1" H 6565 4746 50  0000 L CNN
-F 1 ".1uF" H 6565 4655 50  0000 L CNN
-F 2 "Capacitor_THT:CP_Radial_D5.0mm_P2.00mm" H 6450 4700 50  0001 C CNN
-F 3 "~" H 6450 4700 50  0001 C CNN
-	1    6450 4700
-	-1   0    0    -1
-$EndComp
-Connection ~ 6450 4550
-Wire Wire Line
-	6450 4550 6500 4550
-Connection ~ 7150 4550
-Wire Wire Line
-	7150 4550 7200 4550
-$Comp
 L Device:R_Network05 RN2210

Commit message: SPI peripherals routed
Connections:
- net SD_MISO: now also RN2210.5 (R4); no longer RN2210.3 (R2)
- net SD_MOSI: now also RN2210.3 (R2); no longer RN2210.5 (R4)
Changed lines of the file:
@@
 Text Label 8100 4700 0    50   ~ 0
 SD_SCK
-Text Label 8100 4800 0    50   ~ 0
+Text Label 8100 4600 0    50   ~ 0
 SD_MOSI
 Wire Wire Line
 	8100 4700 8450 4700
 Wire Wire Line
-	8100 4800 8450 4800
+	8100 4600 8450 4600
 Wire Wire Line
 	8450 4500 8100 4500
 Text Label 8100 4500 0    50   ~ 0
 SD_CS
-Text Label 8100 4600 0    50   ~ 0
+Text Label 8100 4800 0    50   ~ 0
 SD_MISO
 Wire Wire Line
-	8100 4600 8450 4600
+	8100 4800 8450 4800
 $Comp
 L power:+3.3V #PWR?

Commit message: Design Rule Check
Connections:
- no-connect marks 4 -> 7
Changed lines of the file:
@@
 	0    -1   -1   0
 $EndComp
+NoConn ~ 6150 3450
+NoConn ~ 6150 3550
+NoConn ~ 8450 4900
 $EndSCHEMATC

Commit message: just totally redid the whole thing
Parts:
- added U1: LP2985-3.3, Package_TO_SOT_SMD:SOT-23-5, symbol Regulator_Linear:LP2985-3.3
- C2210: footprint Capacitor_THT:C_Rect_L4.0mm_W2.5mm_P2.50mm -> Capacitor_SMD:C_1206_3216Metric
Connections:
- net GND: now also U1.2 (GND)
- net MISO: now also U2210.2; no longer U2210.6
- net MOSI: now also U2210.5; no longer U2210.1
- net SD_MISO: now also U2210.1; no longer U2210.5
- net SD_MOSI: now also U2210.6; no longer U2210.2
Changed lines of the file:
@@
 $Descr A4 11693 8268
 encoding utf-8
-Sheet 5 9
+Sheet 5 8
 Title ""
 Date ""
@@
 $EndComp
 Wire Wire Line
-	5000 3750 4650 3750
+	5000 2800 4650 2800
 $Comp
 L power:+3.3V #PWR?
@@
 AR Path="/6191B6A2/61F28B7D/625A5E8B" Ref="U?"  Part="1"
 AR Path="/6191B6A2/61F28B7D/62590ED9/625A5E8B" Ref="U2210"  Part="1"
-F 0 "U2210" H 3500 2900 50  0000 C CNN
-F 1 "74LS07" H 3500 2800 50  0000 C CNN
+F 0 "U2210" H 5200 2700 50  0000 C CNN
+F 1 "74LS07" H 5200 2800 50  0000 C CNN
 F 2 "Package_SO:SOIC-14_3.9x8.7mm_P1.27mm" H 4350 2800 50  0001 C CNN
 F 3 "www.ti.com/lit/ds/symlink/sn74ls07.pdf" H 4350 2800 50  0001 C CNN
 	1    4350 2800
-	1    0    0    -1
+	-1   0    0    1
 $EndComp
 $Comp
@@
 AR Path="/6191B6A2/61F28B7D/625A5E97" Ref="U?"  Part="3"
 AR Path="/6191B6A2/61F28B7D/62590ED9/625A5E97" Ref="U2210"  Part="3"
-F 0 "U2210" H 5200 3800 50  0000 C CNN
-F 1 "74LS07" H 5200 3700 50  0000 C CNN
+F 0 "U2210" H 3500 3850 50  0000 C CNN
+F 1 "74LS07" H 3500 3750 50  0000 C CNN
 F 2 "Package_SO:SOIC-14_3.9x8.7mm_P1.27mm" H 4350 3750 50  0001 C CNN
 F 3 "www.ti.com/lit/ds/symlink/sn74ls07.pdf" H 4350 3750 50  0001 C CNN
 	3    4350 3750
-	-1   0    0    1
+	1    0    0    -1
 $EndComp
 $Comp
@@
 	4650 3300 5000 3300
 Wire Wire Line
-	4650 2800 5000 2800
+	4650 3750 5000 3750
 $Comp
 L power:+5V #PWR?
@@
 Text HLabel 4050 2300 0    50   Input ~ 0
 CS
-Text HLabel 4050 2800 0    50   Input ~ 0
+Text HLabel 4050 3750 0    50   Input ~ 0
 MOSI
 Text HLabel 4050 3300 0    50   Input ~ 0
 SCK
-Text HLabel 4050 3750 0    50   Output ~ 0
+Text HLabel 4050 2800 0    50   Output ~ 0
 MISO
 Text Label 5000 2300 2    50   ~ 0
 SD_CS
-Text Label 5000 2800 2    50   ~ 0
+Text Label 5000 3750 2    50   ~ 0
 SD_MOSI
 Text Label 5000 3300 2    50   ~ 0
 SD_SCK
-Text Label 5000 3750 2    50   ~ 0
+Text Label 5000 2800 2    50   ~ 0
 SD_MISO
 Text Notes 7800 6900 0    118  ~ 24
@@
 F 0 "C2210" H 2265 4446 50  0000 L CNN
 F 1 "22pf" H 2265 4355 50  0000 L CNN
-F 2 "Capacitor_THT:C_Rect_L4.0mm_W2.5mm_P2.50mm" H 2188 4250 50  0001 C CNN
+F 2 "Capacitor_SMD:C_1206_3216Metric" H 2188 4250 50  0001 C CNN
 F 3 "~" H 2150 4400 50  0001 C CNN
 	1    2150 4400
@@
 NoConn ~ 6150 3550
 NoConn ~ 8450 4900
+$Comp
+L Regulator_Linear:LP2985-3.3 U1
+U 1 1 62E8B900
+P 4100 6400
+F 0 "U1" H 4100 6742 50  0000 C CNN
+F 1 "LP2985-3.3" H 4100 6651 50  0000 C CNN
+F 2 "Package_TO_SOT_SMD:SOT-23-5" H 4100 6725 50  0001 C CNN
+F 3 "http://www.ti.com/lit/ds/symlink/lp2985.pdf" H 4100 6400 50  0001 C CNN
+	1    4100 6400
+	1    0    0    -1
+$EndComp
+$Comp
+L power:GND #PWR?
+U 1 1 62E8CAC5
+P 4100 6700
+AR Path="/62E8CAC5" Ref="#PWR?"  Part="1"
+AR Path="/62497D60/62E8CAC5" Ref="#PWR?"  Part="1"
+AR Path="/61D852D7/62E8CAC5" Ref="#PWR?"  Part="1"
+AR Path="/6195D2C9/62E8CAC5" Ref="#PWR?"  Part="1"
+AR Path="/6191B6A2/61F28B7D/62590ED9/62E8CAC5" Ref="#PWR0119"  Part="1"
+F 0 "#PWR0119" H 4100 6450 50  0001 C CNN
+F 1 "GND" H 4105 6527 50  0000 C CNN
+F 2 "" H 4100 6700 50  0001 C CNN
+F 3 "" H 4100 6700 50  0001 C CNN
+	1    4100 6700
+	1    0    0    -1
+$EndComp
+$Comp
+L power:+5V #PWR?
+U 1 1 62E8D6CF
+P 3400 6300
+AR Path="/6195D2C9/62E8D6CF" Ref="#PWR?"  Part="1"
+AR Path="/6191B6A2/61F28B7D/62590ED9/62E8D6CF" Ref="#PWR0120"  Part="1"
+F 0 "#PWR0120" H 3400 6150 50  0001 C CNN
+F 1 "+5V" H 3415 6473 50  0000 C CNN
+F 2 "" H 3400 6300 50  0001 C CNN
+F 3 "" H 3400 6300 50  0001 C CNN
+	1    3400 6300
+	0    -1   -1   0
+$EndComp
+$Comp
+L power:+3.3V #PWR?
+U 1 1 62E8E7FD
+P 4800 6300
+AR Path="/6191B6A2/61F28B7D/62E8E7FD" Ref="#PWR?"  Part="1"
+AR Path="/6191B6A2/61F28B7D/62590ED9/62E8E7FD" Ref="#PWR0124"  Part="1"
+F 0 "#PWR0124" H 4800 6150 50  0001 C CNN
+F 1 "+3.3V" V 4815 6428 50  0000 L CNN
+F 2 "" H 4800 6300 50  0001 C CNN
+F 3 "" H 4800 6300 50  0001 C CNN
+	1    4800 6300
+	0    1    1    0
+$EndComp
 $EndSCHEMATC

Commit message: A lot of disorganized changes
Parts:
- renumbered RN2210 to RN1, U2210 to U1, U1 to U2
Changed lines of the file:
@@
 $Descr A4 11693 8268
 encoding utf-8
-Sheet 5 8
+Sheet 7 7
 Title ""
 Date ""
@@
 AR Path="/6191B6A2/61F28B7D/6259F3CE" Ref="J?"  Part="1"
 AR Path="/6191B6A2/61F28B7D/62590ED9/6259F3CE" Ref="J2210"  Part="1"
-F 0 "J2210" H 7000 3867 50  0000 C CNN
+AR Path="/6191B6A2/61EBDADB/636B5B34/6259F3CE" Ref="J1"  Part="1"
+F 0 "J1" H 7000 3867 50  0000 C CNN
 F 1 "Micro_SD_Card_Det" H 7000 3776 50  0000 C CNN
 F 2 "Connector_Card:microSD_HC_Molex_104031-0811" H 9100 3750 50  0001 C CNN
@@
 AR Path="/6191B6A2/61F28B7D/6259F3E5" Ref="#PWR?"  Part="1"
 AR Path="/6191B6A2/61F28B7D/62590ED9/6259F3E5" Ref="#PWR0112"  Part="1"
-F 0 "#PWR0112" H 5800 2900 50  0001 C CNN
+AR Path="/6191B6A2/61EBDADB/636B5B34/6259F3E5" Ref="#PWR0118"  Part="1"
+F 0 "#PWR0118" H 5800 2900 50  0001 C CNN
 F 1 "GND" V 5805 3022 50  0000 R CNN
 F 2 "" H 5800 3150 50  0001 C CNN
@@
 AR Path="/6191B6A2/61F28B7D/6259F3ED" Ref="#PWR?"  Part="1"
 AR Path="/6191B6A2/61F28B7D/62590ED9/6259F3ED" Ref="#PWR0116"  Part="1"
-F 0 "#PWR0116" H 5800 2800 50  0001 C CNN
+AR Path="/6191B6A2/61EBDADB/636B5B34/6259F3ED" Ref="#PWR0119"  Part="1"
+F 0 "#PWR0119" H 5800 2800 50  0001 C CNN
 F 1 "+3.3V" V 5815 3078 50  0000 L CNN
 F 2 "" H 5800 2950 50  0001 C CNN
@@
 AR Path="/6191B6A2/61F28B7D/6259F3FB" Ref="#PWR?"  Part="1"
 AR Path="/6191B6A2/61F28B7D/62590ED9/6259F3FB" Ref="#PWR0117"  Part="1"
-F 0 "#PWR0117" H 8850 4350 50  0001 C CNN
+AR Path="/6191B6A2/61EBDADB/636B5B34/6259F3FB" Ref="#PWR0120"  Part="1"
+F 0 "#PWR0120" H 8850 4350 50  0001 C CNN
 F 1 "+3.3V" V 8865 4628 50  0000 L CNN
 F 2 "" H 8850 4500 50  0001 C CNN
@@
 AR Path="/6191B6A2/61F28B7D/6259F401" Ref="#PWR?"  Part="1"
 AR Path="/6191B6A2/61F28B7D/62590ED9/6259F401" Ref="#PWR0118"  Part="1"
-F 0 "#PWR0118" H 7850 3300 50  0001 C CNN
+AR Path="/6191B6A2/61EBDADB/636B5B34/6259F401" Ref="#PWR0124"  Part="1"
+F 0 "#PWR0124" H 7850 3300 50  0001 C CNN
 F 1 "GND" V 7855 3422 50  0000 R CNN
 F 2 "" H 7850 3550 50  0001 C CNN
@@
 AR Path="/6191B6A2/61F28B7D/625A5E8B" Ref="U?"  Part="1"
 AR Path="/6191B6A2/61F28B7D/62590ED9/625A5E8B" Ref="U2210"  Part="1"
-F 0 "U2210" H 5200 2700 50  0000 C CNN
+AR Path="/6191B6A2/61EBDADB/636B5B34/625A5E8B" Ref="U1"  Part="1"
+F 0 "U1" H 5200 2700 50  0000 C CNN
 F 1 "74LS07" H 5200 2800 50  0000 C CNN
 F 2 "Package_SO:SOIC-14_3.9x8.7mm_P1.27mm" H 4350 2800 50  0001 C CNN
@@
 AR Path="/6191B6A2/61F28B7D/625A5E91" Ref="U?"  Part="2"
 AR Path="/6191B6A2/61F28B7D/62590ED9/625A5E91" Ref="U2210"  Part="2"
-F 0 "U2210" H 3500 3400 50  0000 C CNN
+AR Path="/6191B6A2/61EBDADB/636B5B34/625A5E91" Ref="U1"  Part="2"
+F 0 "U1" H 3500 3400 50  0000 C CNN
 F 1 "74LS07" H 3500 3300 50  0000 C CNN
 F 2 "Package_SO:SOIC-14_3.9x8.7mm_P1.27mm" H 4350 3300 50  0001 C CNN
@@
 AR Path="/6191B6A2/61F28B7D/625A5E97" Ref="U?"  Part="3"
 AR Path="/6191B6A2/61F28B7D/62590ED9/625A5E97" Ref="U2210"  Part="3"
-F 0 "U2210" H 3500 3850 50  0000 C CNN
+AR Path="/6191B6A2/61EBDADB/636B5B34/625A5E97" Ref="U1"  Part="3"
+F 0 "U1" H 3500 3850 50  0000 C CNN
 F 1 "74LS07" H 3500 3750 50  0000 C CNN
 F 2 "Package_SO:SOIC-14_3.9x8.7mm_P1.27mm" H 4350 3750 50  0001 C CNN
@@
 AR Path="/6191B6A2/61F28B7D/625A5E9D" Ref="U?"  Part="4"
 AR Path="/6191B6A2/61F28B7D/62590ED9/625A5E9D" Ref="U2210"  Part="4"
-F 0 "U2210" H 3500 2400 50  0000 C CNN
+AR Path="/6191B6A2/61EBDADB/636B5B34/625A5E9D" Ref="U1"  Part="4"
+F 0 "U1" H 3500 2400 50  0000 C CNN
 F 1 "74LS07" H 3500 2300 50  0000 C CNN
 F 2 "Package_SO:SOIC-14_3.9x8.7mm_P1.27mm" H 4350 2300 50  0001 C CNN
@@
 AR Path="/6191B6A2/61F28B7D/625A5EA3" Ref="U?"  Part="5"
 AR Path="/6191B6A2/61F28B7D/62590ED9/625A5EA3" Ref="U2210"  Part="5"
-F 0 "U2210" H 4500 5517 50  0000 C CNN
+AR Path="/6191B6A2/61EBDADB/636B5B34/625A5EA3" Ref="U1"  Part="5"
+F 0 "U1" H 4500 5517 50  0000 C CNN
 F 1 "74LS07" H 4500 5426 50  0000 C CNN
 F 2 "Package_SO:SOIC-14_3.9x8.7mm_P1.27mm" H 4500 5200 50  0001 C CNN
@@
 AR Path="/6191B6A2/61F28B7D/625A5EA9" Ref="U?"  Part="7"
 AR Path="/6191B6A2/61F28B7D/62590ED9/625A5EA9" Ref="U2210"  Part="7"
-F 0 "U2210" V 4900 4550 50  0000 L CNN
+AR Path="/6191B6A2/61EBDADB/636B5B34/625A5EA9" Ref="U1"  Part="7"
+F 0 "U1" V 4900 4550 50  0000 L CNN
 F 1 "74LS07" V 4800 4550 50  0000 L CNN
 F 2 "Package_SO:SOIC-14_3.9x8.7mm_P1.27mm" H 4500 4650 50  0001 C CNN
@@
 AR Path="/6191B6A2/61F28B7D/625BC2E4" Ref="#PWR?"  Part="1"
 AR Path="/6191B6A2/61F28B7D/62590ED9/625BC2E4" Ref="#PWR0125"  Part="1"
+AR Path="/6191B6A2/61EBDADB/636B5B34/625BC2E4" Ref="#PWR0125"  Part="1"
 F 0 "#PWR0125" H 4000 4500 50  0001 C CNN
 F 1 "+5V" V 4015 4778 50  0000 L CNN
@@
 AR Path="/6191B6A2/61F28B7D/625BCDFC" Ref="#PWR?"  Part="1"
 AR Path="/6191B6A2/61F28B7D/62590ED9/625BCDFC" Ref="#PWR0126"  Part="1"
+AR Path="/6191B6A2/61EBDADB/636B5B34/625BCDFC" Ref="#PWR0126"  Part="1"
 F 0 "#PWR0126" H 5000 4400 50  0001 C CNN
 F 1 "GND" H 5005 4477 50  0000 C CNN
@@
 AR Path="/6195D2C9/62613B08" Ref="C?"  Part="1"
 AR Path="/6191B6A2/61F28B7D/62590ED9/62613B08" Ref="C2210"  Part="1"
-F 0 "C2210" H 2265 4446 50  0000 L CNN
+AR Path="/6191B6A2/61EBDADB/636B5B34/62613B08" Ref="C1"  Part="1"
+F 0 "C1" H 2265 4446 50  0000 L CNN
 F 1 "22pf" H 2265 4355 50  0000 L CNN
 F 2 "Capacitor_SMD:C_1206_3216Metric" H 2188 4250 50  0001 C CNN
@@
 AR Path="/6195D2C9/62613B0E" Ref="#PWR?"  Part="1"
 AR Path="/6191B6A2/61F28B7D/62590ED9/62613B0E" Ref="#PWR0149"  Part="1"
-F 0 "#PWR0149" H 2150 4300 50  0001 C CNN
+AR Path="/6191B6A2/61EBDADB/636B5B34/62613B0E" Ref="#PWR0127"  Part="1"
+F 0 "#PWR0127" H 2150 4300 50  0001 C CNN
 F 1 "GND" H 2155 4377 50  0000 C CNN
 F 2 "" H 2150 4550 50  0001 C CNN
@@
 AR Path="/6195D2C9/62613B14" Ref="#PWR?"  Part="1"
 AR Path="/6191B6A2/61F28B7D/62590ED9/62613B14" Ref="#PWR0150"  Part="1"
-F 0 "#PWR0150" H 2150 4100 50  0001 C CNN
+AR Path="/6191B6A2/61EBDADB/636B5B34/62613B14" Ref="#PWR0128"  Part="1"
+F 0 "#PWR0128" H 2150 4100 50  0001 C CNN
 F 1 "+5V" H 2165 4423 50  0000 C CNN
 F 2 "" H 2150 4250 50  0001 C CNN
@@
 $EndComp
 $Comp
-L Device:R_Network05 RN2210
+L Device:R_Network05 RN1
 U 1 1 62618FEB
 P 8650 4700
-F 0 "RN2210" V 8233 4700 50  0000 C CNN
+F 0 "RN1" V 8233 4700 50  0000 C CNN
 F 1 "10k" V 8324 4700 50  0000 C CNN
 F 2 "Resistor_THT:R_Array_SIP6" V 9025 4700 50  0001 C CNN
@@
 	4650 2300 5000 2300
 $Comp
-L 74xx:74LS07 U2210
+L 74xx:74LS07 U1
 U 6 1 6293BD1C
 P 3450 5200
-F 0 "U2210" H 3450 5500 50  0000 C CNN
+F 0 "U1" H 3450 5500 50  0000 C CNN
 F 1 "74LS07" H 3450 5400 50  0000 C CNN
 F 2 "Package_SO:SOIC-14_3.9x8.7mm_P1.27mm" H 3450 5200 50  0001 C CNN
@@
 AR Path="/6191B6A2/61F28B7D/6293E9E7" Ref="#PWR?"  Part="1"
 AR Path="/6191B6A2/61F28B7D/62590ED9/6293E9E7" Ref="#PWR0146"  Part="1"
-F 0 "#PWR0146" H 3750 5050 50  0001 C CNN
+AR Path="/6191B6A2/61EBDADB/636B5B34/6293E9E7" Ref="#PWR0129"  Part="1"
+F 0 "#PWR0129" H 3750 5050 50  0001 C CNN
 F 1 "+5V" V 3765 5328 50  0000 L CNN
 F 2 "" H 3750 5200 50  0001 C CNN
@@
 AR Path="/6191B6A2/61F28B7D/6281E96A" Ref="#PWR?"  Part="1"
 AR Path="/6191B6A2/61F28B7D/62590ED9/6281E96A" Ref="#PWR0166"  Part="1"
-F 0 "#PWR0166" H 4800 4950 50  0001 C CNN
+AR Path="/6191B6A2/61EBDADB/636B5B34/6281E96A" Ref="#PWR0146"  Part="1"
+F 0 "#PWR0146" H 4800 4950 50  0001 C CNN
 F 1 "GND" H 4805 5027 50  0000 C CNN
 F 2 "" H 4800 5200 50  0001 C CNN
@@
 NoConn ~ 8450 4900
 $Comp
-L Regulator_Linear:LP2985-3.3 U1
+L Regulator_Linear:LP2985-3.3 U2
 U 1 1 62E8B900
 P 4100 6400
-F 0 "U1" H 4100 6742 50  0000 C CNN
+F 0 "U2" H 4100 6742 50  0000 C CNN
 F 1 "LP2985-3.3" H 4100 6651 50  0000 C CNN
 F 2 "Package_TO_SOT_SMD:SOT-23-5" H 4100 6725 50  0001 C CNN
@@
 AR Path="/6195D2C9/62E8CAC5" Ref="#PWR?"  Part="1"
 AR Path="/6191B6A2/61F28B7D/62590ED9/62E8CAC5" Ref="#PWR0119"  Part="1"
-F 0 "#PWR0119" H 4100 6450 50  0001 C CNN
+AR Path="/6191B6A2/61EBDADB/636B5B34/62E8CAC5" Ref="#PWR0147"  Part="1"
+F 0 "#PWR0147" H 4100 6450 50  0001 C CNN
 F 1 "GND" H 4105 6527 50  0000 C CNN
 F 2 "" H 4100 6700 50  0001 C CNN
@@
 AR Path="/6195D2C9/62E8D6CF" Ref="#PWR?"  Part="1"
 AR Path="/6191B6A2/61F28B7D/62590ED9/62E8D6CF" Ref="#PWR0120"  Part="1"
-F 0 "#PWR0120" H 3400 6150 50  0001 C CNN
+AR Path="/6191B6A2/61EBDADB/636B5B34/62E8D6CF" Ref="#PWR0148"  Part="1"
+F 0 "#PWR0148" H 3400 6150 50  0001 C CNN
 F 1 "+5V" H 3415 6473 50  0000 C CNN
 F 2 "" H 3400 6300 50  0001 C CNN
@@
 AR Path="/6191B6A2/61F28B7D/62E8E7FD" Ref="#PWR?"  Part="1"
 AR Path="/6191B6A2/61F28B7D/62590ED9/62E8E7FD" Ref="#PWR0124"  Part="1"
-F 0 "#PWR0124" H 4800 6150 50  0001 C CNN
+AR Path="/6191B6A2/61EBDADB/636B5B34/62E8E7FD" Ref="#PWR0149"  Part="1"
+F 0 "#PWR0149" H 4800 6150 50  0001 C CNN
 F 1 "+3.3V" V 4815 6428 50  0000 L CNN
 F 2 "" H 4800 6300 50  0001 C CNN
