File: V3/kicad/2220_ROM.sch (KiCad schematic (older format))
At the start: 8 parts, among them J2220 AVR-ISP-6, J2221 Conn_01x02_Male, U2220 25LCxxx, U2221 74HCT126

Commit message: routing SD card control signals
Connections:
- net LC_HOLD is gone; now on net PROG_EN: RN2220.5 (R4)
- net PROG_EN: no longer RN2220.6 (R5)
Changed lines of the file:
@@
 Wire Wire Line
 	4200 4500 4700 4500
-Text Label 8900 4950 0    50   ~ 0
+Text Label 8900 4850 0    50   ~ 0
 PROG_EN
 $Comp
@@
 	1    0    0    -1
 $EndComp
-Wire Wire Line
-	9250 4850 8900 4850
-Text Label 8900 4850 0    50   ~ 0
-LC_HOLD
 Connection ~ 6600 5250
 Wire Wire Line
@@
 NoConn ~ 7600 2900
 Wire Wire Line
-	8900 4950 9250 4950
+	8900 4850 9250 4850
 Wire Wire Line
 	6700 5050 6600 5050

Commit message: SPI peripherals routed
Connections:
- net LC_MISO: now also RN2220.3 (R2); no longer RN2220.4 (R3)
- net LC_MOSI: now also RN2220.5 (R4); no longer RN2220.2 (R1)
- net LC_SCK: now also RN2220.4 (R3); no longer RN2220.3 (R2)
- net PROG_EN: now also RN2220.6 (R5); no longer RN2220.5 (R4)
Changed lines of the file:
@@
 	-1   0    0    1
 $EndComp
-Text Label 8900 4550 0    50   ~ 0
+Text Label 8900 4850 0    50   ~ 0
 LC_MOSI
 Wire Wire Line
-	9250 4550 8900 4550
+	9250 4850 8900 4850
+Text Label 8900 4750 0    50   ~ 0
+LC_SCK
+Wire Wire Line
+	9250 4750 8900 4750
 Text Label 8900 4650 0    50   ~ 0
-LC_SCK
+LC_MISO
 Wire Wire Line
 	9250 4650 8900 4650
-Text Label 8900 4750 0    50   ~ 0
-LC_MISO
-Wire Wire Line
-	9250 4750 8900 4750
 $Comp
 L power:+5V #PWR?
@@
 Wire Wire Line
 	4200 4500 4700 4500
-Text Label 8900 4850 0    50   ~ 0
+Text Label 8900 4950 0    50   ~ 0
 PROG_EN
 $Comp
@@
 NoConn ~ 7600 2900
 Wire Wire Line
-	8900 4850 9250 4850
+	8900 4950 9250 4950
 Wire Wire Line
 	6700 5050 6600 5050

Commit message: Design Rule Check
Connections:
- no-connect marks 1 -> 2
Changed lines of the file:
@@
 Wire Wire Line
 	3750 3450 3400 3450
+NoConn ~ 9250 4550
 $EndSCHEMATC
