File: V3/kicad/z80vga.kicad_pcb (KiCad board)
At the start: 2 copper layers, 135 x 100 mm, 58 parts, among them J1000 Barrel_Jack_Switch, J2120 USB_B, J2121 Conn_01x03_Male, J2122 Conn_01x02_Male, J2200 Conn_01x08_Male, J2201 Conn_01x08_Male, J2210 Micro_SD_Card_Det, J2220 AVR-ISP-6, J2221 Conn_01x02_Male, SW2110 SW_Push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

Commit message: totally redid board layout
Parts:
- moved J2121 120.1 mm to (36.0, 94.0)
- moved J1000 117.1 mm to (40.0, 81.0), turned to 0 degrees
- moved J2120 111.2 mm to (42.0, 108.0), turned to 180 degrees
- moved D1000 107.0 mm to (44.0, 71.0), turned to 180 degrees
- moved C2121 95.4 mm to (53.0, 116.0), turned to 180 degrees
- moved C1000 90.7 mm to (54.6, 89.3), turned to 270 degrees
- moved C2120 89.3 mm to (50.0, 98.0)
- moved U2120 89.3 mm to (51.0, 107.0)
- moved C1001 86.3 mm to (62.2, 89.3), turned to 270 degrees
- moved C1002 84.0 mm to (66.0, 62.0)
- moved C1003 84.0 mm to (66.0, 54.0)
- moved U1001 84.0 mm to (56.0, 58.0)
- moved J2210 74.0 mm to (49.0, 38.0)
- moved U1000 74.0 mm to (58.4, 77.8), turned to 90 degrees
- moved R2120 73.6 mm to (59.0, 112.0)
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Routing:
- net /2000_Z80/2100_ALTCPU/RX: track 0.00 -> 75.7 mm, vias 0 -> 2
- net /2000_Z80/2100_ALTCPU/TX: track 0.00 -> 70.6 mm, vias 0 -> 2
- net Net-(J2120-Pad1): track 0.00 -> 15.4 mm
- net Net-(J2120-Pad3): track 0.00 -> 14.4 mm
- net Net-(C2121-Pad1): track 0.00 -> 12.2 mm, vias 0 -> 1
- net Net-(J2120-Pad2): track 0.00 -> 11.9 mm
- net Net-(C1000-Pad1): track 6.18 -> 0.00 mm
- net +5V: track 6.18 -> 0.00 mm
