File: V3/kicad/2110_Reset.sch (KiCad schematic (older format))
At the start: 7 parts, among them SW1000 SW_Push, U1000 LM555xM

Commit message: Design Rule Check
Connections:
- no-connect marks 0 -> 1
Changed lines of the file:
@@
 Wire Wire Line
 	6700 3150 6700 4050
+NoConn ~ 4350 3050
 $EndSCHEMATC

Commit message: just totally redid the whole thing
Parts:
- removed RN2110: 10k, Resistor_THT:R_Array_SIP4, symbol Device:R_Network03
- added R14, R15: R, Resistor_SMD:R_1206_3216Metric, symbol Device:R
- C1000, C1001, C1002, C1003: footprint Capacitor_THT:C_Rect_L4.0mm_W2.5mm_P2.50mm -> Capacitor_SMD:C_1206_3216Metric
Connections:
- net +5V: now also R14.1, R15.2
- net at C1003.1, SW1000.2, U1000.2 (TR): now also R14.2
- net at C1002.1, U1000.6 (THR), U1000.7 (DIS): now also R15.1
- no-connect marks 1 -> 0
Changed lines of the file:
@@
 $Descr A4 11693 8268
 encoding utf-8
-Sheet 8 9
+Sheet 7 8
 Title ""
 Date ""
@@
 F 0 "C2112" H 5115 4596 50  0000 L CNN
 F 1 "10nF" H 5115 4505 50  0000 L CNN
-F 2 "Capacitor_THT:C_Rect_L4.0mm_W2.5mm_P2.50mm" H 5038 4400 50  0001 C CNN
+F 2 "Capacitor_SMD:C_1206_3216Metric" H 5038 4400 50  0001 C CNN
 F 3 "~" H 5000 4550 50  0001 C CNN
 	1    5000 4550
@@
 Wire Wire Line
 	6700 4250 6700 4050
-Connection ~ 6700 4050
 $Comp
 L Device:C C?
@@
 F 0 "C2111" H 6815 4596 50  0000 L CNN
 F 1 "10uF" H 6815 4505 50  0000 L CNN
-F 2 "Capacitor_THT:C_Rect_L4.0mm_W2.5mm_P2.50mm" H 6738 4400 50  0001 C CNN
+F 2 "Capacitor_SMD:C_1206_3216Metric" H 6738 4400 50  0001 C CNN
 F 3 "~" H 6700 4550 50  0001 C CNN
 	1    6700 4550
@@
 F 0 "C2110" H 8015 3946 50  0000 L CNN
 F 1 "22pF" H 8015 3855 50  0000 L CNN
-F 2 "Capacitor_THT:C_Rect_L4.0mm_W2.5mm_P2.50mm" H 7938 3750 50  0001 C CNN
+F 2 "Capacitor_SMD:C_1206_3216Metric" H 7938 3750 50  0001 C CNN
 F 3 "~" H 7900 3900 50  0001 C CNN
 	1    7900 3900
@@
 F 0 "C2113" H 4565 4596 50  0000 L CNN
 F 1 "100nF" H 4565 4505 50  0000 L CNN
-F 2 "Capacitor_THT:C_Rect_L4.0mm_W2.5mm_P2.50mm" H 4488 4400 50  0001 C CNN
+F 2 "Capacitor_SMD:C_1206_3216Metric" H 4488 4400 50  0001 C CNN
 F 3 "~" H 4450 4550 50  0001 C CNN
 	1    4450 4550
@@
 Wire Wire Line
 	4450 4400 4450 3850
-Connection ~ 4750 3850
 Text Notes 7850 6900 0    118  ~ 24
 This page has been checked!
-$Comp
-L power:+5V #PWR0103
-U 1 1 61E872A1
-P 3950 3250
-AR Path="/61D852D7/61E872A1" Ref="#PWR0103"  Part="1"
-AR Path="/6191B6A2/624CF3AF/61E872A1" Ref="#PWR?"  Part="1"
-AR Path="/6191B6A2/61EBDADB/62512FB8/61E872A1" Ref="#PWR0108"  Part="1"
-F 0 "#PWR0108" H 3950 3100 50  0001 C CNN
-F 1 "+5V" V 3965 3378 50  0000 L CNN
-F 2 "" H 3950 3250 50  0001 C CNN
-F 3 "" H 3950 3250 50  0001 C CNN
-	1    3950 3250
-	0    -1   -1   0
-$EndComp
 $Comp
 L power:+5V #PWR0104
@@
 Connection ~ 4450 4700
 Wire Wire Line
-	4450 3850 4750 3850
-Wire Wire Line
 	4450 4700 5000 4700
-Wire Wire Line
-	4750 3850 5300 3850
-$Comp
-L Device:R_Network03 RN2110
-U 1 1 6256C4FE
-P 4150 3150
-F 0 "RN2110" V 4450 3000 50  0000 L CNN
-F 1 "10k" V 4350 3100 50  0000 L CNN
-F 2 "Resistor_THT:R_Array_SIP4" V 4425 3150 50  0001 C CNN
-F 3 "http://www.vishay.com/docs/31509/csc.pdf" H 4150 3150 50  0001 C CNN
-	1    4150 3150
+$Comp
+L power:+5V #PWR?
+U 1 1 62F79AB5
+P 7000 4050
+AR Path="/6191B6A2/61EBDADB/62F79AB5" Ref="#PWR?"  Part="1"
+AR Path="/6191B6A2/61EBDADB/62512FB8/62F79AB5" Ref="#PWR0108"  Part="1"
+F 0 "#PWR0108" H 7000 3900 50  0001 C CNN
+F 1 "+5V" V 7015 4178 50  0000 L CNN
+F 2 "" H 7000 4050 50  0001 C CNN
+F 3 "" H 7000 4050 50  0001 C CNN
+	1    7000 4050
+	0    1    1    0
+$EndComp
+$Comp
+L Device:R R?
+U 1 1 62F79ABB
+P 5050 3700
+AR Path="/6191B6A2/61EBDADB/62F79ABB" Ref="R?"  Part="1"
+AR Path="/6191B6A2/61EBDADB/62512FB8/62F79ABB" Ref="R14"  Part="1"
+F 0 "R14" V 4843 3700 50  0000 C CNN
+F 1 "R" V 4934 3700 50  0000 C CNN
+F 2 "Resistor_SMD:R_1206_3216Metric" V 4980 3700 50  0001 C CNN
+F 3 "~" H 5050 3700 50  0001 C CNN
+	1    5050 3700
+	1    0    0    -1
+$EndComp
+$Comp
+L power:+5V #PWR?
+U 1 1 62F79AC1
+P 5050 3550
+AR Path="/6191B6A2/61EBDADB/62F79AC1" Ref="#PWR?"  Part="1"
+AR Path="/6191B6A2/61EBDADB/62512FB8/62F79AC1" Ref="#PWR0155"  Part="1"
+F 0 "#PWR0155" H 5050 3400 50  0001 C CNN
+F 1 "+5V" V 5065 3678 50  0000 L CNN
+F 2 "" H 5050 3550 50  0001 C CNN
+F 3 "" H 5050 3550 50  0001 C CNN
+	1    5050 3550
+	1    0    0    -1
+$EndComp
+Connection ~ 5050 3850
+Wire Wire Line
+	5050 3850 5300 3850
+Wire Wire Line
+	4450 3850 5050 3850
+$Comp
+L Device:R R?
+U 1 1 62F79AAF
+P 6850 4050
+AR Path="/6191B6A2/61EBDADB/62F79AAF" Ref="R?"  Part="1"
+AR Path="/6191B6A2/61EBDADB/62512FB8/62F79AAF" Ref="R15"  Part="1"
+F 0 "R15" V 6643 4050 50  0000 C CNN
+F 1 "R" V 6734 4050 50  0000 C CNN
+F 2 "Resistor_SMD:R_1206_3216Metric" V 6780 4050 50  0001 C CNN
+F 3 "~" H 6850 4050 50  0001 C CNN
+	1    6850 4050
 	0    -1   -1   0
 $EndComp
-Wire Wire Line
-	4350 3250 4750 3250
-Wire Wire Line
-	4750 3250 4750 3850
-Wire Wire Line
-	4350 3150 6700 3150
-Wire Wire Line
-	6700 3150 6700 4050
-NoConn ~ 4350 3050
+Connection ~ 6700 4050
 $EndSCHEMATC
