File: V3/kicad/2110_Reset.sch (KiCad schematic (older format))
At the start: 8 parts, among them SW1000 SW_Push, U1000 LM555xM

Commit message: some footprints re-added to board
Parts:
- R14: value R -> 1M
- R15: value R -> 2111
Changed lines of the file:
@@
 $Descr A4 11693 8268
 encoding utf-8
-Sheet 5 6
+Sheet 4 6
 Title ""
 Date ""
@@
 AR Path="/6191B6A2/61EBDADB/62F79ABB" Ref="R?"  Part="1"
 AR Path="/6191B6A2/61EBDADB/62512FB8/62F79ABB" Ref="R14"  Part="1"
-AR Path="/63A83936/62512FB8/62F79ABB" Ref="R14"  Part="1"
-F 0 "R14" V 4843 3700 50  0000 C CNN
-F 1 "R" V 4934 3700 50  0000 C CNN
+AR Path="/63A83936/62512FB8/62F79ABB" Ref="R2110"  Part="1"
+F 0 "R2110" V 4843 3700 50  0000 C CNN
+F 1 "1M" V 4934 3700 50  0000 C CNN
 F 2 "Resistor_SMD:R_1206_3216Metric" V 4980 3700 50  0001 C CNN
 F 3 "~" H 5050 3700 50  0001 C CNN
@@
 AR Path="/63A83936/62512FB8/62F79AAF" Ref="R15"  Part="1"
 F 0 "R15" V 6643 4050 50  0000 C CNN
-F 1 "R" V 6734 4050 50  0000 C CNN
+F 1 "2111" V 6734 4050 50  0000 C CNN
 F 2 "Resistor_SMD:R_1206_3216Metric" V 6780 4050 50  0001 C CNN
 F 3 "~" H 6850 4050 50  0001 C CNN
