File: V3/kicad/3000_Memory.sch (KiCad schematic (older format))
At the start: 5 parts, among them U3000 28C256, U3001 AS6C8008-55_TSOP, U3002 GAL16V8

Commit message: probably going to split into two boards
Parts:
- C3000, C3001: footprint Capacitor_THT:C_Rect_L7.0mm_W2.5mm_P5.00mm -> Capacitor_THT:C_Rect_L4.0mm_W2.5mm_P2.50mm
Connections:
- net VCC is gone; now on net +5V: C3000.1, C3001.1
- net +5V: now also U3002.20 (VCC)
Changed lines of the file:
@@
 $Descr A4 11693 8268
 encoding utf-8
-Sheet 16 16
+Sheet 10 7
 Title ""
 Date ""
@@
 F 0 "C3000" H 1615 3396 50  0000 L CNN
 F 1 "C" H 1615 3305 50  0000 L CNN
-F 2 "Capacitor_THT:C_Rect_L7.0mm_W2.5mm_P5.00mm" H 1538 3200 50  0001 C CNN
+F 2 "Capacitor_THT:C_Rect_L4.0mm_W2.5mm_P2.50mm" H 1538 3200 50  0001 C CNN
 F 3 "~" H 1500 3350 50  0001 C CNN
 	1    1500 3350
-	1    0    0    -1
-$EndComp
-$Comp
-L power:VCC #PWR?
-U 1 1 61A8BF9A
-P 1500 3200
-AR Path="/61A8BF9A" Ref="#PWR?"  Part="1"
-AR Path="/62497D60/61A8BF9A" Ref="#PWR?"  Part="1"
-AR Path="/61D852D7/61A8BF9A" Ref="#PWR?"  Part="1"
-AR Path="/6195D2C9/61A8BF9A" Ref="#PWR0153"  Part="1"
-F 0 "#PWR0153" H 1500 3050 50  0001 C CNN
-F 1 "VCC" H 1515 3373 50  0000 C CNN
-F 2 "" H 1500 3200 50  0001 C CNN
-F 3 "" H 1500 3200 50  0001 C CNN
-	1    1500 3200
 	1    0    0    -1
 $EndComp
@@
 F 0 "C3001" H 2115 3396 50  0000 L CNN
 F 1 "C" H 2115 3305 50  0000 L CNN
-F 2 "Capacitor_THT:C_Rect_L7.0mm_W2.5mm_P5.00mm" H 2038 3200 50  0001 C CNN
+F 2 "Capacitor_THT:C_Rect_L4.0mm_W2.5mm_P2.50mm" H 2038 3200 50  0001 C CNN
 F 3 "~" H 2000 3350 50  0001 C CNN
 	1    2000 3350
-	1    0    0    -1
-$EndComp
-$Comp
-L power:VCC #PWR?
-U 1 1 61A8DCA5
-P 2000 3200
-AR Path="/61A8DCA5" Ref="#PWR?"  Part="1"
-AR Path="/62497D60/61A8DCA5" Ref="#PWR?"  Part="1"
-AR Path="/61D852D7/61A8DCA5" Ref="#PWR?"  Part="1"
-AR Path="/6195D2C9/61A8DCA5" Ref="#PWR0155"  Part="1"
-F 0 "#PWR0155" H 2000 3050 50  0001 C CNN
-F 1 "VCC" H 2015 3373 50  0000 C CNN
-F 2 "" H 2000 3200 50  0001 C CNN
-F 3 "" H 2000 3200 50  0001 C CNN
-	1    2000 3200
 	1    0    0    -1
 $EndComp
@@
 Text HLabel 8500 4300 0    50   Input ~ 0
 A[0..19]
+$Comp
+L power:+5V #PWR0113
+U 1 1 620096C3
+P 2000 3200
+F 0 "#PWR0113" H 2000 3050 50  0001 C CNN
+F 1 "+5V" H 2015 3373 50  0000 C CNN
+F 2 "" H 2000 3200 50  0001 C CNN
+F 3 "" H 2000 3200 50  0001 C CNN
+	1    2000 3200
+	1    0    0    -1
+$EndComp
+$Comp
+L power:+5V #PWR0114
+U 1 1 62009F7F
+P 1500 3200
+F 0 "#PWR0114" H 1500 3050 50  0001 C CNN
+F 1 "+5V" H 1515 3373 50  0000 C CNN
+F 2 "" H 1500 3200 50  0001 C CNN
+F 3 "" H 1500 3200 50  0001 C CNN
+	1    1500 3200
+	1    0    0    -1
+$EndComp
+$Comp
+L power:+5V #PWR0115
+U 1 1 6200D2FF
+P 9550 3300
+F 0 "#PWR0115" H 9550 3150 50  0001 C CNN
+F 1 "+5V" H 9565 3473 50  0000 C CNN
+F 2 "" H 9550 3300 50  0001 C CNN
+F 3 "" H 9550 3300 50  0001 C CNN
+	1    9550 3300
+	0    1    1    0
+$EndComp
 Wire Bus Line
 	8650 3800 8650 4300

Commit message: Updated PCB files
Parts:
- removed U3000: 28C256, Package_DIP:DIP-28_W15.24mm_LongPads, symbol Memory_EEPROM:28C256
- removed U3001: AS6C8008-55_TSOP, Package_SO:TSOP-II-44_10.16x18.41mm_P0.8mm, symbol as6c8008-55_tsop:AS6C8008-55_TSOP
- removed U3002: GAL16V8, Package_DIP:DIP-20_W7.62mm_Socket_LongPads, symbol Logic_Programmable:GAL16V8
- added U3000: SST39SF040, Package_DIP:DIP-32_W15.24mm_LongPads, symbol Memory_Flash:SST39SF040
- added U3001: AS6C4008-55PCN, Package_SO:TSOP-II-32_21.0x10.2mm_P1.27mm, symbol Memory_RAM:AS6C4008-55PCN
- C3000, C3001: value C -> 22pf
Connections:
- net +5V: now also U3000.31 (PGM), U3000.32 (VCC), U3001.32 (VCC)
- net A0: now also U3000.12 (A0), U3001.12 (A0)
- net A1: now also U3000.11 (A1), U3001.11 (A1)
- net A10: now also U3000.23 (A10), U3001.23 (A10)
- net A11: now also U3000.25 (A11), U3001.25 (A11)
- net A12: now also U3000.4 (A12), U3001.4 (A12)
- net A13: now also U3000.28 (A13), U3001.28 (A13)
- net A14: now also U3000.29 (A14), U3001.3 (A14)
- net A15: now also U3000.3 (A15), U3001.31 (A15)
- net A16: now also U3000.2 (A16), U3001.2 (A16)
- net A17: now also U3000.30 (A17), U3001.30 (A17)
- net A18: now also U3000.1 (A18), U3001.1 (A18)
- net A2: now also U3000.10 (A2), U3001.10 (A2)
- net A3: now also U3000.9 (A3), U3001.9 (A3)
- net A4: now also U3000.8 (A4), U3001.8 (A4)
- net A5: now also U3000.7 (A5), U3001.7 (A5)
- net A6: now also U3000.6 (A6), U3001.6 (A6)
- net A7: now also U3000.5 (A7), U3001.5 (A7)
- net A8: now also U3000.27 (A8), U3001.27 (A8)
- net A9: now also U3000.26 (A9), U3001.26 (A9)
- net D0: now also U3000.13 (D0), U3001.13 (DQ0)
- net D1: now also U3000.14 (D1), U3001.14 (DQ1)
- net D2: now also U3000.15 (D2), U3001.15 (DQ2)
- net D3: now also U3000.17 (D3), U3001.17 (DQ3)
- net D4: now also U3000.18 (D4), U3001.18 (DQ4)
- net D5: now also U3000.19 (D5), U3001.19 (DQ5)
- net D6: now also U3000.20 (D6), U3001.20 (DQ6)
- net D7: now also U3000.21 (D7), U3001.21 (DQ7)
- net GND: now also U3000.16 (GND), U3001.16 (VSS)
- net RAM_CS: now also U3001.22 (CE#)
- net READ: now also U3000.24 (OE), U3001.24 (OE#)
- net ROM_CS: now also U3000.22 (CE)
- new net WRITE: U3001.29 (WE#)
Other:
- note added: "This page has been checked!"
- note removed: "This page has NOT been checked!"
- moved on the sheet: C3000, C3001

Commit message: last touches on peripherals and memory
Other:
- moved on the sheet: U3001
Changed lines of the file:
@@
 $EndDescr
 Entry Wire Line
-	5700 2850 5800 2950
-Entry Wire Line
-	5700 2950 5800 3050
-Entry Wire Line
-	5700 3050 5800 3150
-Entry Wire Line
-	5700 3150 5800 3250
-Entry Wire Line
-	5700 3250 5800 3350
-Entry Wire Line
-	5700 3350 5800 3450
-Entry Wire Line
-	5700 3450 5800 3550
-Entry Wire Line
-	5700 3550 5800 3650
-Wire Wire Line
-	5800 2950 6100 2950
-Wire Wire Line
-	5800 3050 6100 3050
-Wire Wire Line
-	5800 3150 6100 3150
-Wire Wire Line
-	5800 3250 6100 3250
-Wire Wire Line
-	5800 3350 6100 3350
-Wire Wire Line
-	5800 3450 6100 3450
-Wire Wire Line
-	5800 3550 6100 3550
-Wire Wire Line
-	5800 3650 6100 3650
-Entry Wire Line
-	5700 3650 5800 3750
-Entry Wire Line
-	5700 3750 5800 3850
-Entry Wire Line
-	5700 3850 5800 3950
-Entry Wire Line
-	5700 3950 5800 4050
-Entry Wire Line
-	5700 4050 5800 4150
-Entry Wire Line
-	5700 4150 5800 4250
-Entry Wire Line
-	5700 4250 5800 4350
-Wire Wire Line
-	5800 3750 6100 3750
-Wire Wire Line
-	5800 3850 6100 3850
-Wire Wire Line
-	5800 3950 6100 3950
-Wire Wire Line
-	5800 4050 6100 4050
-Wire Wire Line
-	5800 4150 6100 4150
-Wire Wire Line
-	5800 4250 6100 4250
-Wire Wire Line
-	5800 4350 6100 4350
-Text Label 5850 2950 0    50   ~ 0
+	5700 2900 5800 3000
+Entry Wire Line
+	5700 3000 5800 3100
+Entry Wire Line
+	5700 3100 5800 3200
+Entry Wire Line
+	5700 3200 5800 3300
+Entry Wire Line
+	5700 3300 5800 3400
+Entry Wire Line
+	5700 3400 5800 3500
+Entry Wire Line
+	5700 3500 5800 3600
+Entry Wire Line
+	5700 3600 5800 3700
+Wire Wire Line
+	5800 3000 6100 3000
+Wire Wire Line
+	5800 3100 6100 3100
+Wire Wire Line
+	5800 3200 6100 3200
+Wire Wire Line
+	5800 3300 6100 3300
+Wire Wire Line
+	5800 3400 6100 3400
+Wire Wire Line
+	5800 3500 6100 3500
+Wire Wire Line
+	5800 3600 6100 3600
+Wire Wire Line
+	5800 3700 6100 3700
+Entry Wire Line
+	5700 3700 5800 3800
+Entry Wire Line
+	5700 3800 5800 3900
+Entry Wire Line
+	5700 3900 5800 4000
+Entry Wire Line
+	5700 4000 5800 4100
+Entry Wire Line
+	5700 4100 5800 4200
+Entry Wire Line
+	5700 4200 5800 4300
+Entry Wire Line
+	5700 4300 5800 4400
+Wire Wire Line
+	5800 3800 6100 3800
+Wire Wire Line
+	5800 3900 6100 3900
+Wire Wire Line
+	5800 4000 6100 4000
+Wire Wire Line
+	5800 4100 6100 4100
+Wire Wire Line
+	5800 4200 6100 4200
+Wire Wire Line
+	5800 4300 6100 4300
+Wire Wire Line
+	5800 4400 6100 4400
+Text Label 5850 3000 0    50   ~ 0
 A0
-Text Label 5850 3050 0    50   ~ 0
+Text Label 5850 3100 0    50   ~ 0
 A1
-Text Label 5850 3150 0    50   ~ 0
+Text Label 5850 3200 0    50   ~ 0
 A2
-Text Label 5850 3250 0    50   ~ 0
+Text Label 5850 3300 0    50   ~ 0
 A3
-Text Label 5850 3350 0    50   ~ 0
+Text Label 5850 3400 0    50   ~ 0
 A4
-Text Label 5850 3450 0    50   ~ 0
+Text Label 5850 3500 0    50   ~ 0
 A5
-Text Label 5850 3550 0    50   ~ 0
+Text Label 5850 3600 0    50   ~ 0
 A6
-Text Label 5850 3650 0    50   ~ 0
+Text Label 5850 3700 0    50   ~ 0
 A7
-Text Label 5850 3750 0    50   ~ 0
+Text Label 5850 3800 0    50   ~ 0
 A8
-Text Label 5850 3850 0    50   ~ 0
+Text Label 5850 3900 0    50   ~ 0
 A9
-Text Label 5850 3950 0    50   ~ 0
+Text Label 5850 4000 0    50   ~ 0
 A10
-Text Label 5850 4050 0    50   ~ 0
+Text Label 5850 4100 0    50   ~ 0
 A11
-Text Label 5850 4150 0    50   ~ 0
+Text Label 5850 4200 0    50   ~ 0
 A12
-Text Label 5850 4250 0    50   ~ 0
+Text Label 5850 4300 0    50   ~ 0
 A13
-Text Label 5850 4350 0    50   ~ 0
+Text Label 5850 4400 0    50   ~ 0
 A14
 Entry Wire Line
-	7600 3050 7500 2950
-Entry Wire Line
-	7600 3150 7500 3050
-Entry Wire Line
-	7600 3250 7500 3150
-Entry Wire Line
-	7600 3350 7500 3250
-Entry Wire Line
-	7600 3450 7500 3350
-Entry Wire Line
-	7600 3550 7500 3450
-Entry Wire Line
-	7600 3650 7500 3550
-Entry Wire Line
-	7600 3750 7500 3650
+	7600 3100 7500 3000
+Entry Wire Line
+	7600 3200 7500 3100
+Entry Wire Line
+	7600 3300 7500 3200
+Entry Wire Line
+	7600 3400 7500 3300
+Entry Wire Line
+	7600 3500 7500 3400
+Entry Wire Line
+	7600 3600 7500 3500
+Entry Wire Line
+	7600 3700 7500 3600
+Entry Wire Line
+	7600 3800 7500 3700
 Entry Wire Line
 	5500 3050 5400 2950
@@
 	5500 3750 5400 3650
 Wire Wire Line
-	7100 2950 7500 2950
-Wire Wire Line
-	7100 3050 7500 3050
-Wire Wire Line
-	7100 3150 7500 3150
-Wire Wire Line
-	7100 3250 7500 3250
-Wire Wire Line
-	7100 3350 7500 3350
-Wire Wire Line
-	7100 3450 7500 3450
-Wire Wire Line
-	7100 3550 7500 3550
-Wire Wire Line
-	7100 3650 7500 3650
-Text Label 7400 2950 0    50   ~ 0
+	7100 3000 7500 3000
+Wire Wire Line
+	7100 3100 7500 3100
+Wire Wire Line
+	7100 3200 7500 3200
+Wire Wire Line
+	7100 3300 7500 3300
+Wire Wire Line
+	7100 3400 7500 3400
+Wire Wire Line
+	7100 3500 7500 3500
+Wire Wire Line
+	7100 3600 7500 3600
+Wire Wire Line
+	7100 3700 7500 3700
+Text Label 7400 3000 0    50   ~ 0
 D0
-Text Label 7400 3050 0    50   ~ 0
+Text Label 7400 3100 0    50   ~ 0
 D1
-Text Label 7400 3150 0    50   ~ 0
+Text Label 7400 3200 0    50   ~ 0
 D2
-Text Label 7400 3250 0    50   ~ 0
+Text Label 7400 3300 0    50   ~ 0
 D3
-Text Label 7400 3350 0    50   ~ 0
+Text Label 7400 3400 0    50   ~ 0
 D4
-Text Label 7400 3450 0    50   ~ 0
+Text Label 7400 3500 0    50   ~ 0
 D5
-Text Label 7400 3550 0    50   ~ 0
+Text Label 7400 3600 0    50   ~ 0
 D6
-Text Label 7400 3650 0    50   ~ 0
+Text Label 7400 3700 0    50   ~ 0
 D7
 Wire Wire Line
@@
 P 4400 2850
 F 0 "#PWR0151" H 4400 2700 50  0001 C CNN
-F 1 "+5V" V 4415 2978 50  0000 L CNN
+F 1 "+5V" H 4450 2900 50  0000 L CNN
 F 2 "" H 4400 2850 50  0001 C CNN
 F 3 "" H 4400 2850 50  0001 C CNN
 	1    4400 2850
-	0    1    1    0
+	1    0    0    -1
 $EndComp
 $Comp
@@
 $EndComp
 Entry Wire Line
-	5700 4350 5800 4450
-Entry Wire Line
-	5700 4450 5800 4550
-Entry Wire Line
-	5700 4550 5800 4650
-Entry Wire Line
-	5700 4650 5800 4750
-Wire Wire Line
-	5800 4450 6100 4450
-Wire Wire Line
-	5800 4550 6100 4550
-Wire Wire Line
-	5800 4650 6100 4650
-Wire Wire Line
-	5800 4750 6100 4750
-Text Label 5850 4450 0    50   ~ 0
+	5700 4400 5800 4500
+Entry Wire Line
+	5700 4500 5800 4600
+Entry Wire Line
+	5700 4600 5800 4700
+Entry Wire Line
+	5700 4700 5800 4800
+Wire Wire Line
+	5800 4500 6100 4500
+Wire Wire Line
+	5800 4600 6100 4600
+Wire Wire Line
+	5800 4700 6100 4700
+Wire Wire Line
+	5800 4800 6100 4800
+Text Label 5850 4500 0    50   ~ 0
 A15
-Text Label 5850 4550 0    50   ~ 0
+Text Label 5850 4600 0    50   ~ 0
 A16
-Text Label 5850 4650 0    50   ~ 0
+Text Label 5850 4700 0    50   ~ 0
 A17
-Text Label 5850 4750 0    50   ~ 0
+Text Label 5850 4800 0    50   ~ 0
 A18
 $Comp
 L power:+5V #PWR0180
 U 1 1 61F46407
-P 6600 2750
-F 0 "#PWR0180" H 6600 2600 50  0001 C CNN
-F 1 "+5V" V 6615 2878 50  0000 L CNN
-F 2 "" H 6600 2750 50  0001 C CNN
-F 3 "" H 6600 2750 50  0001 C CNN
-	1    6600 2750
-	0    1    1    0
-$EndComp
-Text HLabel 7100 4150 2    50   Input ~ 0
+P 6600 2800
+F 0 "#PWR0180" H 6600 2650 50  0001 C CNN
+F 1 "+5V" H 6650 2850 50  0000 L CNN
+F 2 "" H 6600 2800 50  0001 C CNN
+F 3 "" H 6600 2800 50  0001 C CNN
+	1    6600 2800
+	1    0    0    -1
+$EndComp
+Text HLabel 7100 4200 2    50   Input ~ 0
 WRITE
 $Comp
 L power:GND #PWR0181
 U 1 1 61F61A4C
-P 6600 4950
-F 0 "#PWR0181" H 6600 4700 50  0001 C CNN
-F 1 "GND" H 6605 4777 50  0000 C CNN
-F 2 "" H 6600 4950 50  0001 C CNN
-F 3 "" H 6600 4950 50  0001 C CNN
-	1    6600 4950
+P 6600 5000
+F 0 "#PWR0181" H 6600 4750 50  0001 C CNN
+F 1 "GND" H 6605 4827 50  0000 C CNN
+F 2 "" H 6600 5000 50  0001 C CNN
+F 3 "" H 6600 5000 50  0001 C CNN
+	1    6600 5000
 	1    0    0    -1
 $EndComp
@@
 L Memory_RAM:AS6C4008-55PCN U3001
 U 1 1 62109604
-P 6600 3850
-F 0 "U3001" H 6600 5131 50  0000 C CNN
-F 1 "AS6C4008-55PCN" H 6600 5040 50  0000 C CNN
-F 2 "Package_SO:TSOP-II-32_21.0x10.2mm_P1.27mm" H 6600 3950 50  0001 C CNN
-F 3 "https://www.digikey.com/en/products/detail/alliance-memory-inc/AS6C4008-55ZIN/4234590" H 6600 3950 50  0001 C CNN
-	1    6600 3850
-	1    0    0    -1
-$EndComp
-Text HLabel 7100 3950 2    50   Input ~ 0
+P 6600 3900
+F 0 "U3001" H 6600 5300 50  0000 C CNN
+F 1 "AS6C4008-55PCN" H 6600 5200 50  0000 C CNN
+F 2 "Package_SO:TSOP-II-32_21.0x10.2mm_P1.27mm" H 6600 4000 50  0001 C CNN
+F 3 "https://www.digikey.com/en/products/detail/alliance-memory-inc/AS6C4008-55ZIN/4234590" H 6600 4000 50  0001 C CNN
+	1    6600 3900
+	1    0    0    -1
+$EndComp
+Text HLabel 7100 4000 2    50   Input ~ 0
 RAM_CS
-Text HLabel 7100 4050 2    50   Input ~ 0
+Text HLabel 7100 4100 2    50   Input ~ 0
 READ
 Text HLabel 3800 5150 0    50   Input ~ 0
@@
 U 1 1 625638C2
 P 4400 4150
-F 0 "U3000" H 4400 5631 50  0000 C CNN
-F 1 "SST39SF040" H 4400 5540 50  0000 C CNN
+F 0 "U3000" H 4400 5750 50  0000 C CNN
+F 1 "SST39SF040" H 4400 5650 50  0000 C CNN
 F 2 "Package_DIP:DIP-32_W15.24mm_LongPads" H 4400 4450 50  0001 C CNN
 F 3 "http://ww1.microchip.com/downloads/en/DeviceDoc/25022B.pdf" H 4400 4450 50  0001 C CNN
@@
 	5500 2400 5500 3750
 Wire Bus Line
-	7600 2400 7600 3750
+	7600 2400 7600 3800
 Wire Bus Line
 	5700 2850 5700 5700

Commit message: changed footprint on RAM chip
Parts:
- U3001: footprint Package_SO:TSOP-II-32_21.0x10.2mm_P1.27mm -> Package_SO:SSOP-32_11.305x20.495mm_P1.27mm
Changed lines of the file:
@@
 F 0 "U3001" H 6600 5300 50  0000 C CNN
 F 1 "AS6C4008-55PCN" H 6600 5200 50  0000 C CNN
-F 2 "Package_SO:TSOP-II-32_21.0x10.2mm_P1.27mm" H 6600 4000 50  0001 C CNN
+F 2 "Package_SO:SSOP-32_11.305x20.495mm_P1.27mm" H 6600 4000 50  0001 C CNN
 F 3 "https://www.digikey.com/en/products/detail/alliance-memory-inc/AS6C4008-55ZIN/4234590" H 6600 4000 50  0001 C CNN
 	1    6600 3900

Commit message: just totally redid the whole thing
Parts:
- C3000, C3001: footprint Capacitor_THT:C_Rect_L4.0mm_W2.5mm_P2.50mm -> Capacitor_SMD:C_1206_3216Metric
Changed lines of the file:
@@
 $Descr A4 11693 8268
 encoding utf-8
-Sheet 2 9
+Sheet 2 8
 Title ""
 Date ""
@@
 F 0 "C3000" H 2365 3346 50  0000 L CNN
 F 1 "22pf" H 2365 3255 50  0000 L CNN
-F 2 "Capacitor_THT:C_Rect_L4.0mm_W2.5mm_P2.50mm" H 2288 3150 50  0001 C CNN
+F 2 "Capacitor_SMD:C_1206_3216Metric" H 2288 3150 50  0001 C CNN
 F 3 "~" H 2250 3300 50  0001 C CNN
 	1    2250 3300
@@
 F 0 "C3001" H 2865 3346 50  0000 L CNN
 F 1 "22pf" H 2865 3255 50  0000 L CNN
-F 2 "Capacitor_THT:C_Rect_L4.0mm_W2.5mm_P2.50mm" H 2788 3150 50  0001 C CNN
+F 2 "Capacitor_SMD:C_1206_3216Metric" H 2788 3150 50  0001 C CNN
 F 3 "~" H 2750 3300 50  0001 C CNN
 	1    2750 3300

Commit message: More rearranging
Connections:
- net READ renamed RD
- net WRITE renamed WR
Changed lines of the file:
@@
 	1    0    0    -1
 $EndComp
-Text HLabel 7100 4200 2    50   Input ~ 0
-WRITE
 $Comp
 L power:GND #PWR0181
@@
 Text HLabel 7100 4000 2    50   Input ~ 0
 RAM_CS
-Text HLabel 7100 4100 2    50   Input ~ 0
-READ
 Text HLabel 3800 5150 0    50   Input ~ 0
 ROM_CS
-Text HLabel 3800 5250 0    50   Input ~ 0
-READ
 Connection ~ 7600 2400
-$Comp
-L Memory_Flash:SST39SF040 U3000
-U 1 1 625638C2
-P 4400 4150
-F 0 "U3000" H 4400 5750 50  0000 C CNN
-F 1 "SST39SF040" H 4400 5650 50  0000 C CNN
-F 2 "Package_DIP:DIP-32_W15.24mm_LongPads" H 4400 4450 50  0001 C CNN
-F 3 "http://ww1.microchip.com/downloads/en/DeviceDoc/25022B.pdf" H 4400 4450 50  0001 C CNN
-	1    4400 4150
-	1    0    0    -1
-$EndComp
 Entry Wire Line
 	3200 2850 3300 2950
@@
 Wire Bus Line
 	3200 5700 5700 5700
+Text HLabel 7100 4100 2    50   Input ~ 0
+RD
+Text HLabel 7100 4200 2    50   Input ~ 0
+WR
+Text HLabel 3800 5250 0    50   Input ~ 0
+RD
 Wire Bus Line
 	5500 2400 5500 3750
@@
 Wire Bus Line
 	3200 2850 3200 5700
+$Comp
+L Memory_Flash:SST39SF040 U3000
+U 1 1 625638C2
+P 4400 4150
+F 0 "U3000" H 4400 5750 50  0000 C CNN
+F 1 "SST39SF040" H 4400 5650 50  0000 C CNN
+F 2 "Package_DIP:DIP-32_W15.24mm_LongPads" H 4400 4450 50  0001 C CNN
+F 3 "http://ww1.microchip.com/downloads/en/DeviceDoc/25022B.pdf" H 4400 4450 50  0001 C CNN
+	1    4400 4150
+	1    0    0    -1
+$EndComp
 $EndSCHEMATC
