File: V3/kicad/2230_SD_Card.sch (KiCad schematic (older format))
At the start: 10 parts, among them J2210 Micro_SD_Card_Det, U2210 74LS07, U2230 74LS07, U2231 LP2985-3.3

Commit message: 3.1 fix sheet hierarchy (#13)
* Fixed Schematic Heirarchy issue

* some footprints re-added to board

* Add footprints added

* Minor changes
Connections:
- net SD_MOSI: now also RN2230.7 (R2.2); no longer RN2230.6 (R3.2)
- net SD_SCK: now also RN2230.6 (R3.2); no longer RN2230.7 (R2.2)
Changed lines of the file:
@@
 $Descr A4 11693 8268
 encoding utf-8
-Sheet 7 7
+Sheet 6 6
 Title ""
 Date ""
@@
 AR Path="/6191B6A2/61F28B7D/62590ED9/6259F3CE" Ref="J2210"  Part="1"
 AR Path="/6191B6A2/61EBDADB/636B5B34/6259F3CE" Ref="J2230"  Part="1"
+AR Path="/63A83936/636B5B34/6259F3CE" Ref="J2230"  Part="1"
 F 0 "J2230" H 7000 3867 50  0000 C CNN
 F 1 "Micro_SD_Card_Det" H 7000 3776 50  0000 C CNN
@@
 AR Path="/6191B6A2/61F28B7D/62590ED9/6259F3E5" Ref="#PWR0112"  Part="1"
 AR Path="/6191B6A2/61EBDADB/636B5B34/6259F3E5" Ref="#PWR0118"  Part="1"
+AR Path="/63A83936/636B5B34/6259F3E5" Ref="#PWR0118"  Part="1"
 F 0 "#PWR0118" H 5800 2900 50  0001 C CNN
 F 1 "GND" V 5805 3022 50  0000 R CNN
@@
 AR Path="/6191B6A2/61F28B7D/62590ED9/6259F3ED" Ref="#PWR0116"  Part="1"
 AR Path="/6191B6A2/61EBDADB/636B5B34/6259F3ED" Ref="#PWR0119"  Part="1"
+AR Path="/63A83936/636B5B34/6259F3ED" Ref="#PWR0119"  Part="1"
 F 0 "#PWR0119" H 5800 2800 50  0001 C CNN
 F 1 "+3.3V" V 5815 3078 50  0000 L CNN
@@
 	0    -1   -1   0
 $EndComp
+Text Label 7350 4600 0    50   ~ 0
+SD_SCK
 Text Label 7350 4700 0    50   ~ 0
-SD_SCK
-Text Label 7350 4600 0    50   ~ 0
 SD_MOSI
 Wire Wire Line
+	7350 4600 7700 4600
+Wire Wire Line
 	7350 4700 7700 4700
-Wire Wire Line
-	7350 4600 7700 4600
 Wire Wire Line
 	7700 4800 7350 4800
@@
 AR Path="/6191B6A2/61F28B7D/62590ED9/6259F3FB" Ref="#PWR0117"  Part="1"
 AR Path="/6191B6A2/61EBDADB/636B5B34/6259F3FB" Ref="#PWR0120"  Part="1"
+AR Path="/63A83936/636B5B34/6259F3FB" Ref="#PWR0120"  Part="1"
 F 0 "#PWR0120" H 8100 4350 50  0001 C CNN
 F 1 "+3.3V" V 8115 4628 50  0000 L CNN
@@
 AR Path="/6191B6A2/61F28B7D/62590ED9/6259F401" Ref="#PWR0118"  Part="1"
 AR Path="/6191B6A2/61EBDADB/636B5B34/6259F401" Ref="#PWR0124"  Part="1"
+AR Path="/63A83936/636B5B34/6259F401" Ref="#PWR0124"  Part="1"
 F 0 "#PWR0124" H 7850 3300 50  0001 C CNN
 F 1 "GND" V 7855 3422 50  0000 R CNN
@@
 AR Path="/6191B6A2/61F28B7D/62590ED9/625A5E8B" Ref="U2210"  Part="1"
 AR Path="/6191B6A2/61EBDADB/636B5B34/625A5E8B" Ref="U2230"  Part="1"
+AR Path="/63A83936/636B5B34/625A5E8B" Ref="U2230"  Part="1"
 F 0 "U2230" H 5200 2700 50  0000 C CNN
 F 1 "74LS07" H 5200 2800 50  0000 C CNN
@@
 AR Path="/6191B6A2/61F28B7D/62590ED9/625A5E91" Ref="U2210"  Part="2"
 AR Path="/6191B6A2/61EBDADB/636B5B34/625A5E91" Ref="U2230"  Part="2"
+AR Path="/63A83936/636B5B34/625A5E91" Ref="U2230"  Part="2"
 F 0 "U2230" H 3500 3400 50  0000 C CNN
 F 1 "74LS07" H 3500 3300 50  0000 C CNN
@@
 AR Path="/6191B6A2/61F28B7D/62590ED9/625A5E97" Ref="U2210"  Part="3"
 AR Path="/6191B6A2/61EBDADB/636B5B34/625A5E97" Ref="U2230"  Part="3"
+AR Path="/63A83936/636B5B34/625A5E97" Ref="U2230"  Part="3"
 F 0 "U2230" H 3500 3850 50  0000 C CNN
 F 1 "74LS07" H 3500 3750 50  0000 C CNN
@@
 AR Path="/6191B6A2/61F28B7D/62590ED9/625A5E9D" Ref="U2210"  Part="4"
 AR Path="/6191B6A2/61EBDADB/636B5B34/625A5E9D" Ref="U2230"  Part="4"
+AR Path="/63A83936/636B5B34/625A5E9D" Ref="U2230"  Part="4"
 F 0 "U2230" H 3500 2400 50  0000 C CNN
 F 1 "74LS07" H 3500 2300 50  0000 C CNN
@@
 AR Path="/6191B6A2/61F28B7D/62590ED9/625A5EA3" Ref="U2210"  Part="5"
 AR Path="/6191B6A2/61EBDADB/636B5B34/625A5EA3" Ref="U2230"  Part="5"
+AR Path="/63A83936/636B5B34/625A5EA3" Ref="U2230"  Part="5"
 F 0 "U2230" H 4500 5517 50  0000 C CNN
 F 1 "74LS07" H 4500 5426 50  0000 C CNN
@@
 AR Path="/6191B6A2/61F28B7D/62590ED9/625A5EA9" Ref="U2210"  Part="7"
 AR Path="/6191B6A2/61EBDADB/636B5B34/625A5EA9" Ref="U2230"  Part="7"
+AR Path="/63A83936/636B5B34/625A5EA9" Ref="U2230"  Part="7"
 F 0 "U2230" V 4900 4550 50  0000 L CNN
 F 1 "74LS07" V 4800 4550 50  0000 L CNN
@@
 AR Path="/6191B6A2/61F28B7D/62590ED9/625BC2E4" Ref="#PWR0125"  Part="1"
 AR Path="/6191B6A2/61EBDADB/636B5B34/625BC2E4" Ref="#PWR0125"  Part="1"
+AR Path="/63A83936/636B5B34/625BC2E4" Ref="#PWR0125"  Part="1"
 F 0 "#PWR0125" H 4000 4500 50  0001 C CNN
 F 1 "+5V" V 4015 4778 50  0000 L CNN
@@
 AR Path="/6191B6A2/61F28B7D/62590ED9/625BCDFC" Ref="#PWR0126"  Part="1"
 AR Path="/6191B6A2/61EBDADB/636B5B34/625BCDFC" Ref="#PWR0126"  Part="1"
+AR Path="/63A83936/636B5B34/625BCDFC" Ref="#PWR0126"  Part="1"
 F 0 "#PWR0126" H 5000 4400 50  0001 C CNN
 F 1 "GND" H 5005 4477 50  0000 C CNN
@@
 AR Path="/6191B6A2/61F28B7D/62590ED9/62613B08" Ref="C2210"  Part="1"
 AR Path="/6191B6A2/61EBDADB/636B5B34/62613B08" Ref="C2230"  Part="1"
+AR Path="/63A83936/636B5B34/62613B08" Ref="C2230"  Part="1"
 F 0 "C2230" H 2265 4446 50  0000 L CNN
 F 1 "22pf" H 2265 4355 50  0000 L CNN
@@
 AR Path="/6191B6A2/61F28B7D/62590ED9/62613B0E" Ref="#PWR0149"  Part="1"
 AR Path="/6191B6A2/61EBDADB/636B5B34/62613B0E" Ref="#PWR0127"  Part="1"
+AR Path="/63A83936/636B5B34/62613B0E" Ref="#PWR0127"  Part="1"
 F 0 "#PWR0127" H 2150 4300 50  0001 C CNN
 F 1 "GND" H 2155 4377 50  0000 C CNN
@@
 AR Path="/6191B6A2/61F28B7D/62590ED9/62613B14" Ref="#PWR0150"  Part="1"
 AR Path="/6191B6A2/61EBDADB/636B5B34/62613B14" Ref="#PWR0128"  Part="1"
+AR Path="/63A83936/636B5B34/62613B14" Ref="#PWR0128"  Part="1"
 F 0 "#PWR0128" H 2150 4100 50  0001 C CNN
 F 1 "+5V" H 2165 4423 50  0000 C CNN
@@
 AR Path="/6191B6A2/61F28B7D/62590ED9/6293E9E7" Ref="#PWR0146"  Part="1"
 AR Path="/6191B6A2/61EBDADB/636B5B34/6293E9E7" Ref="#PWR0129"  Part="1"
+AR Path="/63A83936/636B5B34/6293E9E7" Ref="#PWR0129"  Part="1"
 F 0 "#PWR0129" H 3750 5050 50  0001 C CNN
 F 1 "+5V" V 3765 5328 50  0000 L CNN
@@
 AR Path="/6191B6A2/61F28B7D/62590ED9/6281E96A" Ref="#PWR0166"  Part="1"
 AR Path="/6191B6A2/61EBDADB/636B5B34/6281E96A" Ref="#PWR0146"  Part="1"
+AR Path="/63A83936/636B5B34/6281E96A" Ref="#PWR0146"  Part="1"
 F 0 "#PWR0146" H 4800 4950 50  0001 C CNN
 F 1 "GND" H 4805 5027 50  0000 C CNN
@@
 AR Path="/6191B6A2/61F28B7D/62590ED9/62E8CAC5" Ref="#PWR0119"  Part="1"
 AR Path="/6191B6A2/61EBDADB/636B5B34/62E8CAC5" Ref="#PWR0147"  Part="1"
+AR Path="/63A83936/636B5B34/62E8CAC5" Ref="#PWR0147"  Part="1"
 F 0 "#PWR0147" H 4100 6450 50  0001 C CNN
 F 1 "GND" H 4105 6527 50  0000 C CNN
@@
 AR Path="/6191B6A2/61F28B7D/62590ED9/62E8D6CF" Ref="#PWR0120"  Part="1"
 AR Path="/6191B6A2/61EBDADB/636B5B34/62E8D6CF" Ref="#PWR0148"  Part="1"
+AR Path="/63A83936/636B5B34/62E8D6CF" Ref="#PWR0148"  Part="1"
 F 0 "#PWR0148" H 2500 6150 50  0001 C CNN
 F 1 "+5V" H 2515 6473 50  0000 C CNN
@@
 AR Path="/6191B6A2/61F28B7D/62590ED9/62E8E7FD" Ref="#PWR0124"  Part="1"
 AR Path="/6191B6A2/61EBDADB/636B5B34/62E8E7FD" Ref="#PWR0149"  Part="1"
+AR Path="/63A83936/636B5B34/62E8E7FD" Ref="#PWR0149"  Part="1"
 F 0 "#PWR0149" H 5400 6150 50  0001 C CNN
 F 1 "+3.3V" V 5415 6428 50  0000 L CNN
@@
 AR Path="/6191B6A2/61EBDADB/63922F79" Ref="C?"  Part="1"
 AR Path="/6191B6A2/61EBDADB/636B5B34/63922F79" Ref="C2232"  Part="1"
+AR Path="/63A83936/636B5B34/63922F79" Ref="C2232"  Part="1"
 F 0 "C2232" H 2915 6496 50  0000 L CNN
 F 1 "1 uF" H 2915 6405 50  0000 L CNN
@@
 AR Path="/6191B6A2/61EBDADB/63922F7F" Ref="#PWR?"  Part="1"
 AR Path="/6191B6A2/61EBDADB/636B5B34/63922F7F" Ref="#PWR0159"  Part="1"
+AR Path="/63A83936/636B5B34/63922F7F" Ref="#PWR0159"  Part="1"
 F 0 "#PWR0159" H 2800 6350 50  0001 C CNN
 F 1 "GND" H 2805 6427 50  0000 C CNN
@@
 AR Path="/6191B6A2/61EBDADB/6392682E" Ref="C?"  Part="1"
 AR Path="/6191B6A2/61EBDADB/636B5B34/6392682E" Ref="C2233"  Part="1"
+AR Path="/63A83936/636B5B34/6392682E" Ref="C2233"  Part="1"
 F 0 "C2233" H 5015 6496 50  0000 L CNN
 F 1 "2.2 uF" H 5015 6405 50  0000 L CNN
@@
 AR Path="/6191B6A2/61EBDADB/63926834" Ref="#PWR?"  Part="1"
 AR Path="/6191B6A2/61EBDADB/636B5B34/63926834" Ref="#PWR0163"  Part="1"
+AR Path="/63A83936/636B5B34/63926834" Ref="#PWR0163"  Part="1"
 F 0 "#PWR0163" H 4900 6350 50  0001 C CNN
 F 1 "GND" H 4905 6427 50  0000 C CNN
@@
 AR Path="/6191B6A2/61F28B7D/62590ED9/63929039" Ref="#PWR?"  Part="1"
 AR Path="/6191B6A2/61EBDADB/636B5B34/63929039" Ref="#PWR0166"  Part="1"
+AR Path="/63A83936/636B5B34/63929039" Ref="#PWR0166"  Part="1"
 F 0 "#PWR0166" H 3700 6250 50  0001 C CNN
 F 1 "+5V" H 3715 6573 50  0000 C CNN
@@
 AR Path="/6191B6A2/61EBDADB/6392A4CF" Ref="C?"  Part="1"
 AR Path="/6191B6A2/61EBDADB/636B5B34/6392A4CF" Ref="C2234"  Part="1"
+AR Path="/63A83936/636B5B34/6392A4CF" Ref="C2234"  Part="1"
 F 0 "C2234" H 4765 7096 50  0000 L CNN
 F 1 "10 nF" H 4765 7005 50  0000 L CNN
@@
 AR Path="/6191B6A2/61EBDADB/6392A4D5" Ref="#PWR?"  Part="1"
 AR Path="/6191B6A2/61EBDADB/636B5B34/6392A4D5" Ref="#PWR0167"  Part="1"
+AR Path="/63A83936/636B5B34/6392A4D5" Ref="#PWR0167"  Part="1"
 F 0 "#PWR0167" H 4650 6950 50  0001 C CNN
 F 1 "GND" H 4655 7027 50  0000 C CNN
@@
 AR Path="/6191B6A2/61F28B7D/62590ED9/63932C37" Ref="C?"  Part="1"
 AR Path="/6191B6A2/61EBDADB/636B5B34/63932C37" Ref="C2231"  Part="1"
+AR Path="/63A83936/636B5B34/63932C37" Ref="C2231"  Part="1"
 F 0 "C2231" H 8415 2946 50  0000 L CNN
 F 1 "22pf" H 8415 2855 50  0000 L CNN
@@
 AR Path="/6191B6A2/61F28B7D/62590ED9/63932C3D" Ref="#PWR?"  Part="1"
 AR Path="/6191B6A2/61EBDADB/636B5B34/63932C3D" Ref="#PWR0170"  Part="1"
+AR Path="/63A83936/636B5B34/63932C3D" Ref="#PWR0170"  Part="1"
 F 0 "#PWR0170" H 8300 2800 50  0001 C CNN
 F 1 "GND" H 8305 2877 50  0000 C CNN
@@
 AR Path="/6191B6A2/61F28B7D/62590ED9/63933B58" Ref="#PWR?"  Part="1"
 AR Path="/6191B6A2/61EBDADB/636B5B34/63933B58" Ref="#PWR0173"  Part="1"
+AR Path="/63A83936/636B5B34/63933B58" Ref="#PWR0173"  Part="1"
 F 0 "#PWR0173" H 8300 2600 50  0001 C CNN
 F 1 "+3.3V" H 8300 2900 50  0000 L CNN
