File: V3/kicad/2230_SD_Card.sch (KiCad schematic (older format))
At the start: 9 parts, among them J2210 Micro_SD_Card_Det, U1 74LS07, U2 LP2985-3.3, U2210 74LS07

Commit message: 3 1 1 m memory (#15)
* moved EEPROM files to /old

* Reworking 3.0 board

* changed footprint on RAM chip

* cleared out old memory traces

* started on rerouting

* on to autoroute

* little more cleanup

* more cleanup

* ill let the autoroute do the rest

* reroute complete

* made PQFP leads fatter

* Updated GAL logic

* Design Rule Check

* Minor pcb touch up

* gerber files

* just totally redid the whole thing

* More rearranging

* added a few caps

* Routed ROM and RAM together

* more routing

* more routes

* A lot of disorganized changes

* 3.1 CSIO SPI Bus (#9)

* Updated SPI to use CPU signals

8 bit register chip controls CS lines

* Renamed and added caps to SD page

* Cleanup

* 3.1 Resistor Replacement (#10)

* First two R arrays

* Added one more r array

* added cap for SPI FF

* Extended cpu pads (#12)

* 3.1 fix sheet hierarchy (#13)

* Fixed Schematic Heirarchy issue

* some footprints re-added to board

* Add footprints added

* Minor changes

* 3.1 redraw cpu courtyard (#14)

* moved all crtyd lines to same place in file

* Duplicate lines were causing issues

* Added pin header for SPI lines

* routed last of non-bus lines

* attempted to route memory lines

* Added new symbol and footprint

* CTS0 no longer drives an LED

* Final cleanup before memory routing

* got CTS0 and RTS mixed up

* Removed extra led from board

* Updated signature

* small changes
Parts:
- removed RN1: 10k, Resistor_THT:R_Array_SIP6, symbol Device:R_Network05
- added C2231: 22pf, Capacitor_SMD:C_1206_3216Metric, symbol Device:C
- added RN2230: 4 x 10K, Resistor_SMD:R_Array_Convex_4x1206, symbol Device:R_Pack04
- gave numbers to parts that had none: 3
- renumbered U1 to U2230, U2 to U2231
Connections:
- net +3V3: now also C2231.1, RN2230.1 (R1.1), RN2230.2 (R2.1), RN2230.3 (R3.1), RN2230.4 (R4.1)
- net GND: now also C2231.2
- net SD_CS: now also RN2230.8 (R1.2)
- net SD_MISO: now also RN2230.5 (R4.2)
- net SD_MOSI: now also RN2230.7 (R2.2)
- net SD_SCK: now also RN2230.6 (R3.2)
- no-connect marks 7 -> 6
Other:
- moved on the sheet: C2232
