File: V3/kicad/2120_USB.sch (KiCad schematic (older format))
At the start: 7 parts, among them J2120 USB_B, J2121 Conn_01x03_Male, J2122 Conn_01x02_Male, U2120 MCP2221AxP

Commit message: 3 1 1 m memory (#15)
* moved EEPROM files to /old

* Reworking 3.0 board

* changed footprint on RAM chip

* cleared out old memory traces

* started on rerouting

* on to autoroute

* little more cleanup

* more cleanup

* ill let the autoroute do the rest

* reroute complete

* made PQFP leads fatter

* Updated GAL logic

* Design Rule Check

* Minor pcb touch up

* gerber files

* just totally redid the whole thing

* More rearranging

* added a few caps

* Routed ROM and RAM together

* more routing

* more routes

* A lot of disorganized changes

* 3.1 CSIO SPI Bus (#9)

* Updated SPI to use CPU signals

8 bit register chip controls CS lines

* Renamed and added caps to SD page

* Cleanup

* 3.1 Resistor Replacement (#10)

* First two R arrays

* Added one more r array

* added cap for SPI FF

* Extended cpu pads (#12)

* 3.1 fix sheet hierarchy (#13)

* Fixed Schematic Heirarchy issue

* some footprints re-added to board

* Add footprints added

* Minor changes

* 3.1 redraw cpu courtyard (#14)

* moved all crtyd lines to same place in file

* Duplicate lines were causing issues

* Added pin header for SPI lines

* routed last of non-bus lines

* attempted to route memory lines

* Added new symbol and footprint

* CTS0 no longer drives an LED

* Final cleanup before memory routing

* got CTS0 and RTS mixed up

* Removed extra led from board

* Updated signature

* small changes
Parts:
- removed J2121: Conn_01x03_Male, Connector_PinHeader_2.54mm:PinHeader_1x03_P2.54mm_Vertical, symbol Connector:Conn_01x03_Male
- C2120, C2121: footprint Capacitor_THT:C_Rect_L4.0mm_W2.5mm_P2.50mm -> Capacitor_SMD:C_1206_3216Metric
- R2120: footprint Resistor_THT:R_Axial_DIN0309_L9.0mm_D3.2mm_P2.54mm_Vertical -> Resistor_SMD:R_1206_3216Metric
Connections:
- net +5V: now also J2120.1 (VBUS)
- no-connect marks 2 -> 6
Changed lines of the file:
@@
 $Descr A4 11693 8268
 encoding utf-8
-Sheet 9 9
+Sheet 5 6
 Title ""
 Date ""
@@
 AR Path="/6191B6A2/61EBDADB/6254C2C1" Ref="U?"  Part="1"
 AR Path="/6191B6A2/61EBDADB/62542978/6254C2C1" Ref="U2120"  Part="1"
+AR Path="/63A83936/62542978/6254C2C1" Ref="U2120"  Part="1"
 F 0 "U2120" H 5050 3119 50  0000 R CNN
 F 1 "MCP2221AxP" H 5050 3210 50  0000 R CNN
@@
 AR Path="/6191B6A2/61EBDADB/6254C2C7" Ref="#PWR?"  Part="1"
 AR Path="/6191B6A2/61EBDADB/62542978/6254C2C7" Ref="#PWR0130"  Part="1"
+AR Path="/63A83936/62542978/6254C2C7" Ref="#PWR0130"  Part="1"
 F 0 "#PWR0130" H 5050 4450 50  0001 C CNN
 F 1 "+5V" V 5065 4728 50  0000 L CNN
@@
 AR Path="/6191B6A2/61EBDADB/6254C2CD" Ref="#PWR?"  Part="1"
 AR Path="/6191B6A2/61EBDADB/62542978/6254C2CD" Ref="#PWR0131"  Part="1"
+AR Path="/63A83936/62542978/6254C2CD" Ref="#PWR0131"  Part="1"
 F 0 "#PWR0131" H 5450 4250 50  0001 C CNN
 F 1 "+5V" V 5465 4528 50  0000 L CNN
@@
 AR Path="/6191B6A2/61EBDADB/6254C2D3" Ref="J?"  Part="1"
 AR Path="/6191B6A2/61EBDADB/62542978/6254C2D3" Ref="J2120"  Part="1"
+AR Path="/63A83936/62542978/6254C2D3" Ref="J2120"  Part="1"
 F 0 "J2120" H 6420 3897 50  0000 R CNN
 F 1 "USB_B" H 6420 3988 50  0000 R CNN
@@
 AR Path="/6191B6A2/61EBDADB/6254C2D9" Ref="#PWR?"  Part="1"
 AR Path="/6191B6A2/61EBDADB/62542978/6254C2D9" Ref="#PWR0132"  Part="1"
+AR Path="/63A83936/62542978/6254C2D9" Ref="#PWR0132"  Part="1"
 F 0 "#PWR0132" H 6700 3250 50  0001 C CNN
 F 1 "GND" H 6705 3327 50  0000 C CNN
@@
 L power:+5V #PWR?
 U 1 1 6254C2ED
-P 6150 4200
+P 6350 4200
 AR Path="/6191B6A2/61EBDADB/6254C2ED" Ref="#PWR?"  Part="1"
 AR Path="/6191B6A2/61EBDADB/62542978/6254C2ED" Ref="#PWR0133"  Part="1"
-F 0 "#PWR0133" H 6150 4050 50  0001 C CNN
-F 1 "+5V" V 6165 4328 50  0000 L CNN
-F 2 "" H 6150 4200 50  0001 C CNN
-F 3 "" H 6150 4200 50  0001 C CNN
-	1    6150 4200
+AR Path="/63A83936/62542978/6254C2ED" Ref="#PWR0133"  Part="1"
+F 0 "#PWR0133" H 6350 4050 50  0001 C CNN
+F 1 "+5V" V 6365 4328 50  0000 L CNN
+F 2 "" H 6350 4200 50  0001 C CNN
+F 3 "" H 6350 4200 50  0001 C CNN
+	1    6350 4200
 	0    -1   -1   0
 $EndComp
@@
 AR Path="/6191B6A2/61EBDADB/6254C2F3" Ref="#PWR?"  Part="1"
 AR Path="/6191B6A2/61EBDADB/62542978/6254C2F3" Ref="#PWR0134"  Part="1"
+AR Path="/63A83936/62542978/6254C2F3" Ref="#PWR0134"  Part="1"
 F 0 "#PWR0134" H 5050 3050 50  0001 C CNN
 F 1 "GND" H 5055 3127 50  0001 C TNN
@@
 NoConn ~ 4650 4300
 NoConn ~ 4650 4400
-$Comp
-L Connector:Conn_01x03_Male J?
-U 1 1 6254C2E6
-P 6250 4400
-AR Path="/6191B6A2/61EBDADB/6254C2E6" Ref="J?"  Part="1"
-AR Path="/6191B6A2/61EBDADB/62542978/6254C2E6" Ref="J2121"  Part="1"
-F 0 "J2121" V 6358 4589 50  0000 L CNN
-F 1 "Conn_01x03_Male" H 6358 4590 50  0001 C CNN
-F 2 "Connector_PinHeader_2.54mm:PinHeader_1x03_P2.54mm_Vertical" H 6250 4400 50  0001 C CNN
-F 3 "~" H 6250 4400 50  0001 C CNN
-	1    6250 4400
-	0    -1   -1   0
-$EndComp
-Wire Wire Line
-	6150 4200 6250 4200
-Connection ~ 6150 4200
 Text Notes 1250 6500 0    197  ~ 39
 This page has been checked!
@@
 AR Path="/6191B6A2/61EBDADB/62512FB8/6262DF87" Ref="C?"  Part="1"
 AR Path="/6191B6A2/61EBDADB/62542978/6262DF87" Ref="C2120"  Part="1"
+AR Path="/63A83936/62542978/6262DF87" Ref="C2120"  Part="1"
 F 0 "C2120" H 3065 4096 50  0000 L CNN
 F 1 "22pF" H 3065 4005 50  0000 L CNN
-F 2 "Capacitor_THT:C_Rect_L4.0mm_W2.5mm_P2.50mm" H 2988 3900 50  0001 C CNN
+F 2 "Capacitor_SMD:C_1206_3216Metric" H 2988 3900 50  0001 C CNN
 F 3 "~" H 2950 4050 50  0001 C CNN
 	1    2950 4050
@@
 AR Path="/6191B6A2/61EBDADB/62512FB8/6262DF8D" Ref="#PWR?"  Part="1"
 AR Path="/6191B6A2/61EBDADB/62542978/6262DF8D" Ref="#PWR0160"  Part="1"
+AR Path="/63A83936/62542978/6262DF8D" Ref="#PWR0160"  Part="1"
 F 0 "#PWR0160" H 2950 3950 50  0001 C CNN
 F 1 "GND" H 2955 4027 50  0000 C CNN
@@
 AR Path="/6191B6A2/61EBDADB/62512FB8/6262DF93" Ref="#PWR?"  Part="1"
 AR Path="/6191B6A2/61EBDADB/62542978/6262DF93" Ref="#PWR0161"  Part="1"
+AR Path="/63A83936/62542978/6262DF93" Ref="#PWR0161"  Part="1"
 F 0 "#PWR0161" H 2950 3750 50  0001 C CNN
 F 1 "+5V" V 2965 4028 50  0000 L CNN
@@
 AR Path="/6191B6A2/61EBDADB/62512FB8/6262E8F5" Ref="C?"  Part="1"
 AR Path="/6191B6A2/61EBDADB/62542978/6262E8F5" Ref="C2121"  Part="1"
+AR Path="/63A83936/62542978/6262E8F5" Ref="C2121"  Part="1"
 F 0 "C2121" H 5065 5146 50  0000 L CNN
 F 1 "22pF" H 5065 5055 50  0000 L CNN
-F 2 "Capacitor_THT:C_Rect_L4.0mm_W2.5mm_P2.50mm" H 4988 4950 50  0001 C CNN
+F 2 "Capacitor_SMD:C_1206_3216Metric" H 4988 4950 50  0001 C CNN
 F 3 "~" H 4950 5100 50  0001 C CNN
 	1    4950 5100
@@
 AR Path="/6191B6A2/61EBDADB/62512FB8/6262F07C" Ref="#PWR?"  Part="1"
 AR Path="/6191B6A2/61EBDADB/62542978/6262F07C" Ref="#PWR0162"  Part="1"
+AR Path="/63A83936/62542978/6262F07C" Ref="#PWR0162"  Part="1"
 F 0 "#PWR0162" H 4950 5000 50  0001 C CNN
 F 1 "GND" H 4955 5077 50  0000 C CNN
@@
 AR Path="/6191B6A2/61EBDADB/6278A36E" Ref="#PWR?"  Part="1"
 AR Path="/6191B6A2/61EBDADB/62542978/6278A36E" Ref="#PWR0145"  Part="1"
+AR Path="/63A83936/62542978/6278A36E" Ref="#PWR0145"  Part="1"
 F 0 "#PWR0145" H 4150 3150 50  0001 C CNN
 F 1 "+5V" V 4165 3428 50  0000 L CNN
@@
 F 0 "R2120" H 3850 3500 50  0000 L CNN
 F 1 "100k" H 3850 3400 50  0000 L CNN
-F 2 "Resistor_THT:R_Axial_DIN0309_L9.0mm_D3.2mm_P2.54mm_Vertical" V 4080 3450 50  0001 C CNN
+F 2 "Resistor_SMD:R_1206_3216Metric" V 4080 3450 50  0001 C CNN
 F 3 "~" H 4150 3450 50  0001 C CNN
 	1    4150 3450
@@
 Wire Wire Line
 	4150 3600 4450 3600
+NoConn ~ 4650 3500
+NoConn ~ 4650 3600
+NoConn ~ 4650 3700
+NoConn ~ 4650 3800
 $EndSCHEMATC
